File: Moby/Hardware/Logic_Board/Logic_Board.kicad_sch (KiCad schematic)
At the start: 36 parts, among them J1 SOICbite, J2 USB_C_Receptacle_USB2.0, Q1 IRLML0060TRPBF, U1 RP2040, U2 W25Q64JVZP, Y1 445I23D12M00000

Commit message: silliness
Other:
- note added: "lol michael was here"
Changed lines of the file:
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@@
+    (effects (font (size 1.27 1.27)) (justify left bottom))
+  )
+  (text "lol michael was here" (at 209.55 107.95 0)
     (effects (font (size 1.27 1.27)) (justify left bottom))
   )
