File: Tim/Hardware/Logic_Board/Logic_Board.kicad_sch (KiCad schematic)
At the start: 36 parts, among them J1 SOICbite, J2 USB_C_Receptacle_USB2.0, Q1 IRLML0060TRPBF, U1 RP2040, U2 W25Q64JVZP, Y1 445I23D12M00000

Commit message: Some organization and connectors for external stuffs
Connections:
- net LS1: now reaches U1.2 (GPIO0)
- net Ch.A: now reaches U1.3 (GPIO1)
- net Ch.B: now reaches U1.4 (GPIO2)
- net PWM_MC: now reaches U1.5 (GPIO3)
- no-connect marks 22 -> 17
Changed lines of the file:
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@@
   (no_connect (at 228.6 53.34))
   (no_connect (at 116.84 119.38))
-  (no_connect (at 116.84 50.8))
   (no_connect (at 20.32 134.62))
-  (no_connect (at 116.84 68.58))
   (no_connect (at 20.32 129.54))
   (no_connect (at 116.84 73.66))
@@
   (no_connect (at 116.84 124.46))
   (no_connect (at 116.84 114.3))
-  (no_connect (at 116.84 53.34))
   (no_connect (at 116.84 101.6))
   (no_connect (at 116.84 86.36))
-  (no_connect (at 116.84 58.42))
-  (no_connect (at 116.84 55.88))
   (no_connect (at 116.84 127))
   (no_connect (at 228.6 50.8))
@@
     (effects (font (size 1.27 1.27)) (justify left))
   )
+  (hierarchical_label "LS1" (shape input) (at 116.84 50.8 0) (fields_autoplaced)
+    (effects (font (size 1.27 1.27)) (justify left))
+  )
   (hierarchical_label "QSPI_SD2" (shape input) (at 173.99 119.38 0) (fields_autoplaced)
     (effects (font (size 1.27 1.27)) (justify left))
@@
     (effects (font (size 1.27 1.27)) (justify left))
   )
+  (hierarchical_label "Ch.A" (shape input) (at 116.84 53.34 0) (fields_autoplaced)
+    (effects (font (size 1.27 1.27)) (justify left))
+  )
   (hierarchical_label "QSPI_SD3" (shape input) (at 50.8 63.5 180) (fields_autoplaced)
     (effects (font (size 1.27 1.27)) (justify right))
@@
     (effects (font (size 1.27 1.27)) (justify left))
   )
+  (hierarchical_label "Ch.B" (shape input) (at 116.84 55.88 0) (fields_autoplaced)
+    (effects (font (size 1.27 1.27)) (justify left))
+  )
   (hierarchical_label "SCL" (shape input) (at 116.84 63.5 0) (fields_autoplaced)
     (effects (font (size 1.27 1.27)) (justify left))
@@
     (effects (font (size 1.27 1.27)) (justify left))
   )
+  (hierarchical_label "PWM_MC" (shape input) (at 116.84 58.42 0) (fields_autoplaced)
+    (effects (font (size 1.27 1.27)) (justify left))
+  )
