File: Hardware/Tim/Power/Power.kicad_sch (KiCad schematic)
At the start: 2 parts, among them J1 Conn_01x02_Pin, J2 Conn_01x03_Socket

Commit message: Reduntant board has all the stuff?
Parts:
- removed J2: Conn_01x03_Socket, symbol Connector:Conn_01x03_Socket
Other:
- note added: "For cut circuit"
- note removed: "Motor Controller Connector"
Changed lines of the file:
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@@
 (kicad_sch (version 20230121) (generator eeschema)
   (paper "A4")
-  (polyline (pts (xy 238.76 34.29) (xy 238.76 63.5))
-    (stroke (width 0.254) (type dash))
-  )
-  (wire (pts (xy 209.55 43.18) (xy 209.55 44.45))
-    (stroke (width 0) (type default))
-  )
-  (polyline (pts (xy 199.39 63.5) (xy 238.76 63.5))
-    (stroke (width 0.254) (type dash))
-  )
-  (polyline (pts (xy 199.39 34.29) (xy 238.76 34.29))
-    (stroke (width 0.254) (type dash))
-  )
-  (wire (pts (xy 210.82 43.18) (xy 209.55 43.18))
-    (stroke (width 0) (type default))
-  )
-  (polyline (pts (xy 199.39 34.29) (xy 199.39 63.5))
-    (stroke (width 0.254) (type dash))
-  )
-  (text "Motor Controller\nConnector" (at 199.39 63.5 0)
-    (effects (font (size 2 2) (thickness 1.016) bold) (justify left bottom))
-  )
-  (hierarchical_label "PWM_MC" (shape input) (at 210.82 38.1 180) (fields_autoplaced)
-    (effects (font (size 1.27 1.27)) (justify right))
+  (text "For cut circuit" (at 151.13 33.02 0)
+    (effects (font (size 1.27 1.27)) (justify left bottom))
   )
   (symbol (lib_id "power:+3V3") (at 134.62 39.37 0) (unit 1)
@@
     )
   )
-  (symbol (lib_id "Connector:Conn_01x03_Socket") (at 215.9 40.64 0) (unit 1)
-    (in_bom yes) (on_board yes) (dnp no) (fields_autoplaced)
-    (property "Reference" "J2" (at 217.17 39.37 0)
-      (effects (font (size 1.27 1.27)) (justify left))
-    )
-    (property "Value" "Conn_01x03_Socket" (at 217.17 41.91 0)
-      (effects (font (size 1.27 1.27)) (justify left))
-    )
-    (property "Footprint" "" (at 215.9 40.64 0)
-      (effects (font (size 1.27 1.27)) hide)
-    )
-    (property "Datasheet" "~" (at 215.9 40.64 0)
-      (effects (font (size 1.27 1.27)) hide)
-    )
-    (pin "1")
-    (pin "2")
-    (pin "3")
-    (instances
-      (project "Power"
-        (path "/bc4c0cf2-b0a0-4f0a-926b-530333fe541b"
-          (reference "J2") (unit 1)
-        )
-      )
-    )
-  )
   (symbol (lib_id "power:VBUS") (at 55.88 39.37 0) (unit 1)
     (in_bom yes) (on_board yes) (dnp no) (fields_autoplaced)
@@
     )
   )
-  (symbol (lib_id "power:GND") (at 209.55 44.45 0) (unit 1)
+  (symbol (lib_id "power:+BATT") (at 156.21 39.37 0) (unit 1)
     (in_bom yes) (on_board yes) (dnp no) (fields_autoplaced)
-    (property "Reference" "#PWR02" (at 209.55 50.8 0)
+    (property "Reference" "#PWR02" (at 156.21 43.18 0)
       (effects (font (size 1.27 1.27)) hide)
     )
-    (property "Value" "GND" (at 209.55 49.53 0)
+    (property "Value" "+BATT" (at 156.21 34.29 0)
       (effects (font (size 1.27 1.27)))
     )
-    (property "Footprint" "" (at 209.55 44.45 0)
+    (property "Footprint" "" (at 156.21 39.37 0)
       (effects (font (size 1.27 1.27)) hide)
     )
-    (property "Datasheet" "" (at 209.55 44.45 0)
+    (property "Datasheet" "" (at 156.21 39.37 0)
       (effects (font (size 1.27 1.27)) hide)
     )

Commit message: Added color sensors disconnected GPIO in muxing crisis
Other:
- note removed: "For cut circuit"
Changed lines of the file:
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@@
 (kicad_sch (version 20230121) (generator eeschema)
   (paper "A4")
-  (text "For cut circuit" (at 151.13 33.02 0)
-    (effects (font (size 1.27 1.27)) (justify left bottom))
-  )
   (symbol (lib_id "power:+3V3") (at 134.62 39.37 0) (unit 1)
     (in_bom yes) (on_board yes) (dnp no) (fields_autoplaced)
@@
     )
   )
-  (symbol (lib_id "power:+1V1") (at 115.57 39.37 0) (unit 1)
-    (in_bom yes) (on_board yes) (dnp no) (fields_autoplaced)
-    (property "Reference" "#PWR05" (at 115.57 43.18 0)
-      (effects (font (size 1.27 1.27)) hide)
-    )
-    (property "Value" "+1V1" (at 115.57 34.29 0)
-      (effects (font (size 1.27 1.27)))
-    )
-    (property "Footprint" "" (at 115.57 39.37 0)
-      (effects (font (size 1.27 1.27)) hide)
-    )
-    (property "Datasheet" "" (at 115.57 39.37 0)
-      (effects (font (size 1.27 1.27)) hide)
-    )
-    (pin "1")
-    (instances
-      (project "Power"
-        (path "/bc4c0cf2-b0a0-4f0a-926b-530333fe541b"
-          (reference "#PWR05") (unit 1)
-        )
-      )
-    )
-  )
   (symbol (lib_id "power:VBUS") (at 55.88 39.37 0) (unit 1)
     (in_bom yes) (on_board yes) (dnp no) (fields_autoplaced)
@@
         (path "/bc4c0cf2-b0a0-4f0a-926b-530333fe541b"
           (reference "#PWR07") (unit 1)
-        )
-      )
-    )
-  )
-  (symbol (lib_id "power:+BATT") (at 156.21 39.37 0) (unit 1)
-    (in_bom yes) (on_board yes) (dnp no) (fields_autoplaced)
-    (property "Reference" "#PWR02" (at 156.21 43.18 0)
-      (effects (font (size 1.27 1.27)) hide)
-    )
-    (property "Value" "+BATT" (at 156.21 34.29 0)
-      (effects (font (size 1.27 1.27)))
-    )
-    (property "Footprint" "" (at 156.21 39.37 0)
-      (effects (font (size 1.27 1.27)) hide)
-    )
-    (property "Datasheet" "" (at 156.21 39.37 0)
-      (effects (font (size 1.27 1.27)) hide)
-    )
-    (pin "1")
-    (instances
-      (project "Power"
-        (path "/bc4c0cf2-b0a0-4f0a-926b-530333fe541b"
-          (reference "#PWR02") (unit 1)
-        )
-      )
-    )
-  )
-  (symbol (lib_id "power:+1V8") (at 127 39.37 0) (unit 1)
-    (in_bom yes) (on_board yes) (dnp no) (fields_autoplaced)
-    (property "Reference" "#PWR04" (at 127 43.18 0)
-      (effects (font (size 1.27 1.27)) hide)
-    )
-    (property "Value" "+1V8" (at 127 34.29 0)
-      (effects (font (size 1.27 1.27)))
-    )
-    (property "Footprint" "" (at 127 39.37 0)
-      (effects (font (size 1.27 1.27)) hide)
-    )
-    (property "Datasheet" "" (at 127 39.37 0)
-      (effects (font (size 1.27 1.27)) hide)
-    )
-    (pin "1")
-    (instances
-      (project "Power"
-        (path "/bc4c0cf2-b0a0-4f0a-926b-530333fe541b"
-          (reference "#PWR04") (unit 1)
         )
       )
@@
         )
       )
-    )
-  )
-  (symbol (lib_id "power:+1V8") (at 120.65 39.37 0) (unit 1)
-    (in_bom yes) (on_board yes) (dnp no) (fields_autoplaced)
-    (property "Reference" "#PWR06" (at 120.65 43.18 0)
-      (effects (font (size 1.27 1.27)) hide)
-    )
-    (property "Value" "+1V8" (at 120.65 34.29 0)
-      (effects (font (size 1.27 1.27)))
-    )
-    (property "Footprint" "" (at 120.65 39.37 0)
-      (effects (font (size 1.27 1.27)) hide)
-    )
-    (property "Datasheet" "" (at 120.65 39.37 0)
-      (effects (font (size 1.27 1.27)) hide)
-    )
-    (pin "1")
-    (instances
-      (project "Power"
-        (path "/bc4c0cf2-b0a0-4f0a-926b-530333fe541b"
-          (reference "#PWR06") (unit 1)
-        )
-      )
