File: Hardware/Tim/Logic_Board/Logic_Board.kicad_sch (KiCad schematic)
At the start: 36 parts, among them J1 SOICbite, J2 USB_C_Receptacle_USB2.0, Q1 IRLML0060TRPBF, U1 RP2040, U2 W25Q64JVZP, Y1 445I23D12M00000

Commit message: Reduntant board has all the stuff?
Connections:
- net D1: now also U1.11 (GPIO8); no longer U1.8 (GPIO6)
- net PWM_MC: now also U1.7 (GPIO5); no longer U1.5 (GPIO3)
- net SCL: now also U1.9 (GPIO7); no longer U1.7 (GPIO5)
- net SDA: now also U1.8 (GPIO6); no longer U1.6 (GPIO4)
- net Ch.A renamed Ch.1A
- net Ch.B renamed Ch.1B
- new net Ch.2A: U1.5 (GPIO3)
- new net Ch.2B: U1.6 (GPIO4)
- no-connect marks 17 -> 16
Changed lines of the file:
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@@
   (no_connect (at 116.84 121.92))
   (no_connect (at 20.32 132.08))
-  (no_connect (at 116.84 71.12))
   (no_connect (at 116.84 88.9))
   (no_connect (at 116.84 124.46))
@@
     (effects (font (size 1.27 1.27)) (justify left))
   )
-  (hierarchical_label "SDA" (shape input) (at 116.84 60.96 0) (fields_autoplaced)
+  (hierarchical_label "SDA" (shape input) (at 116.84 66.04 0) (fields_autoplaced)
     (effects (font (size 1.27 1.27)) (justify left))
   )
@@
     (effects (font (size 1.27 1.27)) (justify left))
   )
-  (hierarchical_label "Ch.A" (shape input) (at 116.84 53.34 0) (fields_autoplaced)
+  (hierarchical_label "Ch.1A" (shape input) (at 116.84 53.34 0) (fields_autoplaced)
+    (effects (font (size 1.27 1.27)) (justify left))
+  )
+  (hierarchical_label "Ch.2B" (shape input) (at 116.84 60.96 0) (fields_autoplaced)
     (effects (font (size 1.27 1.27)) (justify left))
   )
@@
     (effects (font (size 1.27 1.27)) (justify left))
   )
-  (hierarchical_label "D1" (shape input) (at 116.84 66.04 0) (fields_autoplaced)
+  (hierarchical_label "D1" (shape input) (at 116.84 71.12 0) (fields_autoplaced)
     (effects (font (size 1.27 1.27)) (justify left))
   )
@@
     (effects (font (size 1.27 1.27)) (justify left))
   )
-  (hierarchical_label "Ch.B" (shape input) (at 116.84 55.88 0) (fields_autoplaced)
-    (effects (font (size 1.27 1.27)) (justify left))
-  )
-  (hierarchical_label "SCL" (shape input) (at 116.84 63.5 0) (fields_autoplaced)
+  (hierarchical_label "Ch.1B" (shape input) (at 116.84 55.88 0) (fields_autoplaced)
+    (effects (font (size 1.27 1.27)) (justify left))
+  )
+  (hierarchical_label "SCL" (shape input) (at 116.84 68.58 0) (fields_autoplaced)
+    (effects (font (size 1.27 1.27)) (justify left))
+  )
+  (hierarchical_label "Ch.2A" (shape input) (at 116.84 58.42 0) (fields_autoplaced)
     (effects (font (size 1.27 1.27)) (justify left))
   )
@@
     (effects (font (size 1.27 1.27)) (justify left))
   )
-  (hierarchical_label "PWM_MC" (shape input) (at 116.84 58.42 0) (fields_autoplaced)
-    (effects (font (size 1.27 1.27)) (justify left))
-  )
+  (hierarchical_label "PWM_MC" (shape input) (at 116.84 63.5 0) (fields_autoplaced)
+    (effects (font (size 1.27 1.27)) (justify left))
+  )

Commit message: Added color sensors disconnected GPIO in muxing crisis
Connections:
- net Ch.1A: no longer U1.3 (GPIO1)
- net Ch.1B: no longer U1.4 (GPIO2)
- net Ch.2A: no longer U1.5 (GPIO3)
- net Ch.2B: no longer U1.6 (GPIO4)
- net D1: no longer U1.11 (GPIO8)
- net GPS_RX: no longer U1.15 (GPIO12)
- net GPS_TX: no longer U1.16 (GPIO13)
- net LS1: no longer U1.2 (GPIO0)
- net PWM_MC: no longer U1.7 (GPIO5)
- net SCL: no longer U1.9 (GPIO7)
- net SPI0_MISO: no longer U1.27 (GPIO16)
- net SPI0_MOSI: no longer U1.30 (GPIO19)
- net SPI0_SCK: no longer U1.29 (GPIO18)
- net SW: no longer U1.14 (GPIO11)
- net TXEN: no longer U1.13 (GPIO10)
- net SDA: no longer names the net of U1.8 (GPIO6)
- net SPI0_CS: no longer names the net of U1.28 (GPIO17)
- no-connect marks 16 -> 13
Other:
- note added: "1.1v is internally regualted by rp2040 outputting at VREG_OUT"
- note added: "Encoder circuitry? Missing 1 encoder"
- note added: "These are not connected in the correct order for RP2040 muxing"
Changed lines of the file:
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@@
   (no_connect (at 20.32 134.62))
   (no_connect (at 20.32 129.54))
-  (no_connect (at 116.84 73.66))
   (no_connect (at 116.84 121.92))
   (no_connect (at 20.32 132.08))
-  (no_connect (at 116.84 88.9))
   (no_connect (at 116.84 124.46))
   (no_connect (at 116.84 114.3))
   (no_connect (at 116.84 101.6))
-  (no_connect (at 116.84 86.36))
   (no_connect (at 116.84 127))
   (no_connect (at 228.6 50.8))
@@
     (effects (font (size 1.27 1.27)) (justify left bottom))
   )
+  (text "Encoder circuitry?\nMissing 1 encoder" (at 129.54 60.96 0)
+    (effects (font (size 1.27 1.27)) (justify left bottom))
+  )
+  (text "These are not connected in\nthe correct order for RP2040 muxing"
+    (at 129.54 82.55 0)
+    (effects (font (size 1.27 1.27)) (justify left bottom))
+  )
   (text "This resistor \nensures that \nwe don't \noverdrive \nthe LED"
     (at 173.99 50.8 0)
@@
     (effects (font (size 1.27 1.27)) (justify right bottom))
   )
+  (text "1.1v is internally\nregualted by rp2040\noutputting at VREG_OUT"
+    (at 68.58 17.78 0)
+    (effects (font (size 1.27 1.27) (color 255 0 0 1)) (justify left bottom))
+  )
   (label "SWCLK" (at 49.53 121.92 180) (fields_autoplaced)
     (effects (font (size 1.27 1.27)) (justify right bottom))
@@
     (effects (font (size 1.27 1.27)) (justify right bottom))
   )
-  (hierarchical_label "SW" (shape input) (at 116.84 78.74 0) (fields_autoplaced)
-    (effects (font (size 1.27 1.27)) (justify left))
-  )
-  (hierarchical_label "SDA" (shape input) (at 116.84 66.04 0) (fields_autoplaced)
+  (hierarchical_label "SW" (shape input) (at 119.38 78.74 0) (fields_autoplaced)
+    (effects (font (size 1.27 1.27)) (justify left))
+  )
+  (hierarchical_label "SDA_PT" (shape input) (at 119.38 66.04 0) (fields_autoplaced)
     (effects (font (size 1.27 1.27)) (justify left))
   )
@@
     (effects (font (size 1.27 1.27)) (justify left))
   )
-  (hierarchical_label "SPI0_SCK" (shape input) (at 116.84 96.52 0) (fields_autoplaced)
+  (hierarchical_label "SPI0_SCK" (shape input) (at 119.38 96.52 0) (fields_autoplaced)
     (effects (font (size 1.27 1.27)) (justify left))
   )
@@
     (effects (font (size 1.27 1.27)) (justify left))
   )
-  (hierarchical_label "LS1" (shape input) (at 116.84 50.8 0) (fields_autoplaced)
+  (hierarchical_label "LS1" (shape input) (at 119.38 50.8 0) (fields_autoplaced)
     (effects (font (size 1.27 1.27)) (justify left))
   )
@@
     (effects (font (size 1.27 1.27)) (justify right))
   )
-  (hierarchical_label "GPS_TX" (shape input) (at 116.84 83.82 0) (fields_autoplaced)
+  (hierarchical_label "GPS_TX" (shape input) (at 119.38 83.82 0) (fields_autoplaced)
     (effects (font (size 1.27 1.27)) (justify left))
   )
@@
     (effects (font (size 1.27 1.27)) (justify left))
   )
-  (hierarchical_label "Ch.1A" (shape input) (at 116.84 53.34 0) (fields_autoplaced)
-    (effects (font (size 1.27 1.27)) (justify left))
-  )
-  (hierarchical_label "Ch.2B" (shape input) (at 116.84 60.96 0) (fields_autoplaced)
+  (hierarchical_label "Ch.1A" (shape input) (at 119.38 53.34 0) (fields_autoplaced)
+    (effects (font (size 1.27 1.27)) (justify left))
+  )
+  (hierarchical_label "Ch.2B" (shape input) (at 119.38 60.96 0) (fields_autoplaced)
     (effects (font (size 1.27 1.27)) (justify left))
   )
@@
     (effects (font (size 1.27 1.27)) (justify left))
   )
-  (hierarchical_label "D1" (shape input) (at 116.84 71.12 0) (fields_autoplaced)
-    (effects (font (size 1.27 1.27)) (justify left))
-  )
-  (hierarchical_label "SPI0_MISO" (shape input) (at 116.84 91.44 0) (fields_autoplaced)
+  (hierarchical_label "D1" (shape input) (at 119.38 73.66 0) (fields_autoplaced)
+    (effects (font (size 1.27 1.27)) (justify left))
+  )
+  (hierarchical_label "SPI0_MISO" (shape input) (at 119.38 91.44 0) (fields_autoplaced)
     (effects (font (size 1.27 1.27)) (justify left))
   )
@@
     (effects (font (size 1.27 1.27)) (justify right))
   )
-  (hierarchical_label "SPI0_CS" (shape input) (at 116.84 93.98 0) (fields_autoplaced)
-    (effects (font (size 1.27 1.27)) (justify left))
-  )
-  (hierarchical_label "Ch.1B" (shape input) (at 116.84 55.88 0) (fields_autoplaced)
-    (effects (font (size 1.27 1.27)) (justify left))
-  )
-  (hierarchical_label "SCL" (shape input) (at 116.84 68.58 0) (fields_autoplaced)
-    (effects (font (size 1.27 1.27)) (justify left))
-  )
-  (hierarchical_label "Ch.2A" (shape input) (at 116.84 58.42 0) (fields_autoplaced)
-    (effects (font (size 1.27 1.27)) (justify left))
-  )
-  (hierarchical_label "GPS_RX" (shape input) (at 116.84 81.28 0) (fields_autoplaced)
-    (effects (font (size 1.27 1.27)) (justify left))
-  )
-  (hierarchical_label "SPI0_MOSI" (shape input) (at 116.84 99.06 0) (fields_autoplaced)
+  (hierarchical_label "SPI0_CS_RAD" (shape input) (at 119.38 93.98 0) (fields_autoplaced)
+    (effects (font (size 1.27 1.27)) (justify left))
+  )
+  (hierarchical_label "Ch.1B" (shape input) (at 119.38 55.88 0) (fields_autoplaced)
+    (effects (font (size 1.27 1.27)) (justify left))
+  )
+  (hierarchical_label "SCL" (shape input) (at 119.38 71.12 0) (fields_autoplaced)
+    (effects (font (size 1.27 1.27)) (justify left))
+  )
+  (hierarchical_label "SPIO_CS_IMU" (shape input) (at 119.38 88.9 0) (fields_autoplaced)
+    (effects (font (size 1.27 1.27)) (justify left))
+  )
+  (hierarchical_label "Ch.2A" (shape input) (at 119.38 58.42 0) (fields_autoplaced)
+    (effects (font (size 1.27 1.27)) (justify left))
+  )
+  (hierarchical_label "GPS_RX" (shape input) (at 119.38 81.28 0) (fields_autoplaced)
+    (effects (font (size 1.27 1.27)) (justify left))
+  )
+  (hierarchical_label "SPI0_MOSI" (shape input) (at 119.38 99.06 0) (fields_autoplaced)
     (effects (font (size 1.27 1.27)) (justify left))
   )
@@
     (effects (font (size 1.27 1.27)) (justify left))
   )
-  (hierarchical_label "TXEN" (shape input) (at 116.84 76.2 0) (fields_autoplaced)
+  (hierarchical_label "TXEN" (shape input) (at 119.38 76.2 0) (fields_autoplaced)
+    (effects (font (size 1.27 1.27)) (justify left))
+  )
+  (hierarchical_label "SDA_CLR" (shape input) (at 119.38 68.58 0) (fields_autoplaced)
     (effects (font (size 1.27 1.27)) (justify left))
   )
@@
     (effects (font (size 1.27 1.27)) (justify left))
   )
-  (hierarchical_label "PWM_MC" (shape input) (at 116.84 63.5 0) (fields_autoplaced)
-    (effects (font (size 1.27 1.27)) (justify left))
-  )
+  (hierarchical_label "PWM_MC" (shape input) (at 119.38 63.5 0) (fields_autoplaced)
+    (effects (font (size 1.27 1.27)) (justify left))
+  )
