File: Hardware/Tim/Main board/Main board.kicad_sch (KiCad schematic)
At the start: 119 parts, among them J1 Conn_01x02_Socket, J1 SOICbite, J2 Conn_01x05_Socket, J2 USB_C_Receptacle_USB2.0, J3 Conn_01x04_Socket, J4 Conn_01x03_Socket, J4 Conn_01x04_Socket, J4 Nichrome, J4 U.FL, J5 Conn_01x04_Socket, Q1 IRLML0060TRPBF, U1 BMI270, U1 LT3120JV-PBF, U1 RP2040, U2 W25Q64JVZP, U6 MS5607-02BA, U8 DRF1262TL, Y1 445I23D12M00000, Y2 32.768k

Commit message: routing started
Parts:
- removed C43: 100nF, Capacitor_SMD:C_0603_1608Metric, symbol Device:C_Small
- removed C8: 1uF, PCM_Resistor_SMD_AKL:R_0603_1608Metric_Pad0.98x0.95mm_HandSolder, symbol Device:C_Small
- removed J2: Conn_01x05_Socket, symbol Connector:Conn_01x05_Socket
- removed R30, R31: 0, Resistor_SMD:R_0402_1005Metric, symbol Device:R_Small
- removed U10: ~, Rudolph_Lib:MIA-M10Q, symbol Terminator_Lib:MIA-M10Q
- removed Y2: 32.768k, Crystal:Crystal_SMD_3215-2Pin_3.2x1.5mm, symbol Device:Crystal_Small
- added C19, C20, C45, C46, C49, C50, C53, C54, C55, C56: 1uF, Capacitor_SMD:C_0402_1005Metric, symbol Device:C
- added C47, C48, C51, C52: 1nF, Capacitor_SMD:C_0402_1005Metric, symbol Device:C
- added C7: 10uF, Capacitor_SMD:C_0603_1608Metric, symbol Device:C_Small
- added J1: Conn_01x02_Socket, Connector_Molex:Molex_SL_171971-0002_1x02_P2.54mm_Vertical, symbol Connector:Conn_01x02_Socket
- added J14, J16: Conn_01x02_Pin, Connector_Molex:Molex_SL_171971-0002_1x02_P2.54mm_Vertical, symbol Connector:Conn_01x02_Pin
- added R12: 10k, Resistor_SMD:R_0402_1005Metric, symbol Device:R_Small
- added R15, R16: 0, Resistor_SMD:R_0402_1005Metric, symbol Device:R
- added R32, R33, R34, R35, R36, R37, R38, R39, R40, R41, R42, R43: 100k, Resistor_SMD:R_0402_1005Metric, symbol Device:R
- added R45, R58: 63.4k, Resistor_SMD:R_0402_1005Metric, symbol Device:R
- added R46, R55: 18.2k, Resistor_SMD:R_0402_1005Metric, symbol Device:R
- added R47, R48, R50, R52, R54, R56, R60, R62: 5k, Resistor_SMD:R_0402_1005Metric, symbol Device:R
- added R49, R57: 21.5k, Resistor_SMD:R_0402_1005Metric, symbol Device:R
- added R51, R59: 23.7k, Resistor_SMD:R_0402_1005Metric, symbol Device:R
- added R53, R61: 10.2k, Resistor_SMD:R_0402_1005Metric, symbol Device:R
- added U10: MAX-M10S, RF_GPS:ublox_MAX, symbol RF_GPS:MAX-M10S
- added U11, U13: ADP7105ACPZ-5.0-R7, Package_CSP:LFCSP-8-1EP_3x3mm_P0.5mm_EP1.6x2.34mm, symbol BPP_Lib:ADP7105ACPZ-5.0-R7
- added U12, U5: ADP7105ACPZ-3.3-R7, Package_CSP:LFCSP-8-1EP_3x3mm_P0.5mm_EP1.6x2.34mm, symbol BPP_Lib:ADP7105ACPZ-3.3-R7
- added U14, U15: TPS2121RUXR, BPPlib:TPS2121, symbol BPP_Lib:TPS2121RUXR
- BT1: footprint Rudolph_Lib:SEIKO_ML414H_IV01E -> BPPlib:SEIKO_ML414H_IV01E
- C1, C2: value 100 nF -> 100nF; footprint (none) -> Capacitor_SMD:C_0402_1005Metric
- D1: footprint PCM_Package_TO_SOT_SMD_AKL:SOT-23-6 -> Package_TO_SOT_SMD:TSOT-23-6_HandSoldering
- J1: footprint (none) -> Connector_Molex:Molex_SL_171971-0002_1x02_P2.54mm_Vertical
- J1: footprint Rudolph_Lib:SOIC_clipProgSmall -> BPPlib:SOIC_clipProgSmall
- J3, J4, J5: footprint (none) -> Connector_Molex:Molex_SL_171971-0004_1x04_P2.54mm_Vertical
- J4: footprint (none) -> Connector_Molex:Molex_SL_171971-0003_1x03_P2.54mm_Vertical
- U1: footprint Rudolph_Lib:RP2040-QFN-56 -> BPPlib:RP2040-QFN-56
- U1: footprint Terminator_Lib:LQFN28_Rev0_ADI-M -> Extra Footprints:LQFN28_Rev0_ADI
- U1: footprint BMI270_BOS -> Package_LGA:LGA-14_3x2.5mm_P0.5mm_LayoutBorder3x4y
- U2: footprint Rudolph_Lib:W25Q64JVZP -> Package_SON:WSON-8-1EP_6x5mm_P1.27mm_EP3.4x4.3mm
- U8: footprint Rudolph_Lib:DRF1262TL -> BPPlib:DRF1262TL
Connections:
- net +3.3V is gone; now on net +3V3: C1.1, C10.1, C11.1, C12.1, C13.1, C14.1, C15.1, C2.2, C6.1, C7.1, C8.1, C9.1, J1.1 (Pin_1), JP2.1 (A), R2.1, R8.1, R9.1, U1.1 (IOVDD), U1.10 (IOVDD), U1.22 (IOVDD), U1.33 (IOVDD), U1.42 (IOVDD), U1.43 (ADC_AVDD), U1.44 (VREG_IN), U1.48 (USB_VDD), U1.49 (IOVDD), U1.5 (VDDIO), U1.8 (VDD), U2.8 (VCC)
- net +5P is gone; now on net +5V: J4.1 (Pin_1)
- net +3V3: now also C19.1, C49.1, R12.1, R32.1, R38.1, U10.7 (VCC_IO), U10.8 (VCC), U12.1 (VOUT), U12.2 (SENSE), U5.1 (VOUT), U5.2 (SENSE)
- net +5V: now also C20.1, C50.1, R33.1, R39.1, U11.1 (VOUT), U11.2 (SENSE), U13.1 (VOUT), U13.2 (SENSE)
- net CUT: now also U1.14 (GPIO11); no longer U1.11 (GPIO8)
- net D1: now also U1.11 (GPIO8); no longer Q1.1 (G)
- net GND: now also C19.2, C20.2, C45.2, C46.2, C47.2, C48.2, C49.2, C50.2, C51.2, C52.2, C53.2, C54.2, C55.1, C56.1, C7.2, J14.2 (Pin_2), J16.2 (Pin_2), R34.1, R36.1, R40.1, R41.1, R47.1, R48.1, R49.2, R50.1, R52.1, R54.1, R56.1, R57.2, R60.1, R62.1, U10.1 (GND), U10.10 (GND), U10.12 (GND), U11.3 (GND), U11.6 (GND), U11.9 (GND), U12.3 (GND), U12.6 (GND), U12.9 (GND), U13.3 (GND), U13.6 (GND), U13.9 (GND), U14.12 (GND), U14.9 (ST), U15.12 (GND), U15.9 (ST), U5.3 (GND), U5.6 (GND), U5.9 (GND)
- net LS1: now also U1.17 (GPIO14), R12.2
- net PWM_ART: now also U1.13 (GPIO10)
- net PWM_EMRG_REL: now also U1.13 (GPIO10); no longer U1.9 (GPIO7)
- net PWM_MC: now also U1.14 (GPIO11)
- net SPIO_CS_IMU: now also U1.12 (GPIO9); no longer U1.6 (GPIO4)
- net VBUS: now also R51.2, R53.2, U14.2 (IN2)
- net VCC: now also R59.2, R61.2, U15.2 (IN2)
- net V_BCKP: now also C7.1, U10.6 (V_BCKP)
- net D-: now reaches D1.4 (L2), J2.A7 (D-), J2.B7 (D-)
- net D+: now reaches D1.6 (L1), J2.A6 (D+), J2.B6 (D+)
- net at R22.2: now also J1.1 (Pin_1), U10.3 (RXD)
- net at R21.2: now also J1.2 (Pin_2), U10.2 (TXD)
- net CROSS_PRIMTX_REDRX: now reaches U1.12 (GPIO9)
- net CROSS_PRIMTX_REDRX: now also R15.2
- net at AE1.1 (A): now also U10.11 (RF_IN)
- net EXTINT: now reaches U1.38 (GPIO26_ADC0)
- net EXTINT: now also U10.5 (EXTINT)
- net TIMEPULSE: now reaches U1.39 (GPIO27_ADC1)
- net TIMEPULSE: now also U10.4 (TIMEPULSE)
- net at U1.7 (GPIO5): now also R16.1
- new net: R59.1, R60.2, U15.4 (OV2)
- new net: C51.1, U12.4 (SS)
- new net: R40.2, R43.1, U12.5 (EN/UVLO)
- new net: R38.2, U12.7 (PG)
- new net: C53.1, C54.1, R42.2, R43.2, U12.8 (VIN), U13.8 (VIN), U15.1 (OUT), U15.8 (OUT)
- new net: R55.1, R56.2, U15.6 (PR1)
- new net: C56.2, U15.11 (SS)
- new net: R34.2, R35.1, U11.5 (EN/UVLO)
- new net: C45.1, C46.1, R35.2, R37.2, U11.8 (VIN), U14.1 (OUT), U14.8 (OUT), U5.8 (VIN)
- new net: R36.2, R37.1, U5.5 (EN/UVLO)
- new net: J16.1 (Pin_1), R55.2, R58.2, U15.7 (IN1)
- new net: R49.1, U14.10 (ILM)
- new net: R50.2, R51.1, U14.4 (OV2)
- new net: C48.1, U5.4 (SS)
- new net: R32.2, U5.7 (PG)
- new net: R46.1, R48.2, U14.6 (PR1)
- new net: R52.2, R53.1, U14.3 (CP2)
- new net: R54.2, R58.1, U15.5 (OV1)
- new net: R33.2, U11.7 (PG)
- new net: R39.2, U13.7 (PG)
- new net: C52.1, U13.4 (SS)
- new net: R61.1, R62.2, U15.3 (CP2)
- new net: R41.2, R42.1, U13.5 (EN/UVLO)
- new net: C47.1, U11.4 (SS)
- new net: R57.1, U15.10 (ILM)
- new net: J14.1 (Pin_1), R45.2, R46.2, U14.7 (IN1)
- new net: R45.1, R47.2, U14.5 (OV1)
- new net: C55.2, U14.11 (SS)
- new net: R15.1, U1.6 (GPIO4)
- new net CROSS_PRIMRX_REDTX: R16.2, U1.11 (GPIO8)
- new net D1_R: Q1.1 (G), U1.9 (GPIO7)
- no-connect marks 56 -> 47
Other:
- note added: "Dan mentioned circuitry to convert to step and direction for encoders. Shipman mention 0 cpu time programing options"
- note added: "Footprint for connectors is for vertial version but hole size and spacing is the same"
- note added: "Power"
- note added: "Redundant Power"
- note added: "Resistors can be adjusted to adjust enable disable thresholds"
- note added: "Shipman is currently testing"
- note added: "This muxing work needs to be doubled checked by someone sane"
- note removed: "3v3 is for standard system 3.3v is for redundant"
- note removed: "Color Sensor Connector"
- note removed: "Dan mentioned circuitry to convert to step and direction for encoders"
- note removed: "Encoder circuitry?"
- note removed: "This muxing work needs to be doubled checked by someone sane Needs cross chip comms"
- note removed: "Was this circuit ever tested? How does one power this? Its a short high current?"
- moved on the sheet: AE1, C7, J1, J4, R21, R22, U8

Commit message: Routing donish maybe
Parts:
- U1: footprint Extra Footprints:LQFN28_Rev0_ADI -> BPPlib:LQFN28_Rev0_ADI
Connections:
- net SPIO_PICO is gone; now on net SPI0_PICO: U1.14 (SDX)
- net SPIO_POCI is gone; now on net SPI0_POCI: U1.1 (SDO)
- net SPIO_SCK is gone; now on net SPI0_SCK: U1.13 (SCX)
- net SWCLK: no longer J1.3 (Pin_3), U1.24 (SWCLK)
- net SWD: no longer J1.2 (Pin_2), U1.25 (SWD)
- net +1V1: no longer names the net of C3.1, C4.1, C5.1, U1.23 (DVDD), U1.45 (VREG_VOUT), U1.50 (DVDD)
- net +1V1: no longer C3.1, C4.1, C5.1, U1.23 (DVDD), U1.45 (VREG_VOUT), U1.50 (DVDD)
- new net: C3.1, C4.1, C5.1, U1.23 (DVDD), U1.45 (VREG_VOUT), U1.50 (DVDD)
- new net SWCLK_R: J1.3 (Pin_3), U1.24 (SWCLK)
- new net SWD_R: J1.2 (Pin_2), U1.25 (SWD)
Changed lines of the file:
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@@
   (junction (at 496.57 111.76) (diameter 0) (color 0 0 0 0)
   )
+  (junction (at 63.5 21.59) (diameter 0) (color 0 0 0 0)
+  )
   (junction (at 147.32 114.3) (diameter 0) (color 0 0 0 0)
   )
@@
   (junction (at 60.96 367.03) (diameter 0) (color 0 0 0 0)
   )
-  (junction (at 63.5 21.59) (diameter 0) (color 0 0 0 0)
-  )
   (junction (at 64.77 367.03) (diameter 0) (color 0 0 0 0)
   )
@@
     (stroke (width 0.254) (type dash))
   )
-  (wire (pts (xy 63.5 20.32) (xy 63.5 21.59))
-    (stroke (width 0) (type default))
-  )
   (wire (pts (xy 116.84 208.28) (xy 116.84 214.63))
     (stroke (width 0) (type default))
@@
     (stroke (width 0) (type default))
   )
-  (wire (pts (xy 412.75 21.59) (xy 412.75 22.86))
-    (stroke (width 0) (type default))
-  )
   (wire (pts (xy 125.73 370.84) (xy 134.62 370.84))
     (stroke (width 0) (type default))
@@
     (stroke (width 0) (type default))
   )
+  (wire (pts (xy 63.5 21.59) (xy 66.04 21.59))
+    (stroke (width 0) (type default))
+  )
   (wire (pts (xy 96.52 21.59) (xy 100.33 21.59))
     (stroke (width 0) (type default))
@@
     (stroke (width 0) (type default))
   )
-  (wire (pts (xy 189.23 198.12) (xy 187.96 198.12))
-    (stroke (width 0) (type default))
-  )
   (wire (pts (xy 149.86 41.91) (xy 149.86 43.18))
     (stroke (width 0) (type default))
@@
     (stroke (width 0) (type default))
   )
-  (wire (pts (xy 66.04 21.59) (xy 63.5 21.59))
-    (stroke (width 0) (type default))
-  )
   (wire (pts (xy 82.55 31.75) (xy 82.55 21.59))
     (stroke (width 0) (type default))
@@
     (effects (font (size 1.27 1.27)) (justify right bottom))
   )
-  (label "SWD" (at 398.78 120.65 180) (fields_autoplaced)
+  (label "SWD_R" (at 398.78 120.65 180) (fields_autoplaced)
     (effects (font (size 1.27 1.27)) (justify right bottom))
   )
-  (label "SWCLK" (at 398.78 123.19 180) (fields_autoplaced)
+  (label "SWCLK_R" (at 398.78 123.19 180) (fields_autoplaced)
     (effects (font (size 1.27 1.27)) (justify right bottom))
   )
@@
     (effects (font (size 1.27 1.27)) (justify left))
   )
+  (hierarchical_label "SPI0_SCK" (shape input) (at 229.87 200.66 0) (fields_autoplaced)
+    (effects (font (size 1.27 1.27)) (justify left))
+  )
   (hierarchical_label "QSPI_SCLK" (shape input) (at 50.8 67.31 180) (fields_autoplaced)
     (effects (font (size 1.27 1.27)) (justify right))
@@
     (effects (font (size 1.27 1.27)) (justify left))
   )
+  (hierarchical_label "SPI0_POCI" (shape input) (at 189.23 198.12 180) (fields_autoplaced)
+    (effects (font (size 1.27 1.27)) (justify right))
+  )
   (hierarchical_label "Ch.3B" (shape input) (at 116.84 101.6 0) (fields_autoplaced)
     (effects (font (size 1.27 1.27)) (justify left))
@@
     (effects (font (size 1.27 1.27)) (justify left))
   )
+  (hierarchical_label "SPI0_PICO" (shape input) (at 229.87 198.12 0) (fields_autoplaced)
+    (effects (font (size 1.27 1.27)) (justify left))
+  )
   (hierarchical_label "SW" (shape input) (at 116.84 106.68 0) (fields_autoplaced)
     (effects (font (size 1.27 1.27)) (justify left))
@@
     (effects (font (size 1.27 1.27)) (justify right))
   )
-  (hierarchical_label "SPIO_PICO" (shape input) (at 229.87 198.12 0) (fields_autoplaced)
-    (effects (font (size 1.27 1.27)) (justify left))
-  )
   (hierarchical_label "D1" (shape input) (at 116.84 71.12 0) (fields_autoplaced)
     (effects (font (size 1.27 1.27)) (justify left))
@@
     (effects (font (size 1.27 1.27)) (justify left))
   )
-  (hierarchical_label "SPIO_SCK" (shape input) (at 229.87 200.66 0) (fields_autoplaced)
-    (effects (font (size 1.27 1.27)) (justify left))
-  )
   (hierarchical_label "CROSS_PRIMRX_REDTX" (shape input) (at 466.09 72.39 0) (fields_autoplaced)
     (effects (font (size 1.27 1.27)) (justify left))
@@
     (effects (font (size 1.27 1.27)) (justify left))
   )
-  (hierarchical_label "SPIO_POCI" (shape input) (at 187.96 198.12 180) (fields_autoplaced)
-    (effects (font (size 1.27 1.27)) (justify right))
-  )
   (hierarchical_label "CROSS_PRIMRX_REDTX" (shape input) (at 132.08 63.5 0) (fields_autoplaced)
     (effects (font (size 1.27 1.27)) (justify left))
@@
     )
   )
-  (symbol (lib_id "power:+1V1") (at 412.75 21.59 0) (unit 1)
-    (in_bom yes) (on_board yes) (dnp no)
-    (property "Reference" "#PWR010" (at 412.75 25.4 0)
-      (effects (font (size 1.27 1.27)) hide)
-    )
-    (property "Value" "+1V1" (at 412.75 17.78 0)
-      (effects (font (size 1.27 1.27)))
-    )
-    (property "Footprint" "" (at 412.75 21.59 0)
-      (effects (font (size 1.27 1.27)) hide)
-    )
-    (property "Datasheet" "" (at 412.75 21.59 0)
-      (effects (font (size 1.27 1.27)) hide)
-    )
-    (pin "1")
-    (instances
-      (project "Logic_Board"
-        (path "/02d89edf-b12c-4e48-a419-0665a4b8b6d0"
-          (reference "#PWR010") (unit 1)
-        )
-      )
-      (project "T1000"
-        (path "/12aa2e34-1e28-4012-9c9f-3fbc422880b2"
-          (reference "#PWR012") (unit 1)
-        )
-      )
-      (project "Rudolph_Tracker"
-        (path "/131b2a79-e29c-42e9-9adf-d7be6c6c28ff"
-          (reference "#PWR010") (unit 1)
-        )
-      )
-      (project "Redundant_System"
-        (path "/26e62c7f-f27c-4940-85ae-9c569ff0337a"
-          (reference "#PWR07") (unit 1)
-        )
-      )
-      (project "SLAPS_Solar_Harvester"
-        (path "/65c91e2c-c4db-441a-a788-9bcdc306326f"
-          (reference "#PWR0107") (unit 1)
-        )
-      )
-      (project "BPP_Logger"
-        (path "/974c48bf-534e-4335-98e1-b0426c783e99"
-          (reference "#PWR06") (unit 1)
-        )
-      )
-      (project "GPS_Tracker"
-        (path "/b438986c-8622-4db9-bd4a-ee46786798d0"
-          (reference "#PWR010") (unit 1)
-        )
-      )
-      (project "Main board"
-        (path "/be354753-d7ed-4d26-938b-99a92979eaa8"
-          (reference "#PWR056") (unit 1)
-        )
-      )
-    )
-  )
   (symbol (lib_id "Device:R_Small") (at 232.41 30.48 90) (unit 1)
     (in_bom yes) (on_board yes) (dnp no)
@@
       (effects (font (size 1.524 1.524) bold))
     )
-    (property "Footprint" "Extra Footprints:LQFN28_Rev0_ADI" (at 402.59 251.46 0)
+    (property "Footprint" "BPPlib:LQFN28_Rev0_ADI" (at 402.59 251.46 0)
       (effects (font (size 1.27 1.27) italic) hide)
     )
@@
         )
       )
-    )
-  )
-  (symbol (lib_id "power:+1V1") (at 63.5 20.32 0) (unit 1)
-    (in_bom yes) (on_board yes) (dnp no)
-    (property "Reference" "#PWR010" (at 63.5 24.13 0)
-      (effects (font (size 1.27 1.27)) hide)
-    )
-    (property "Value" "+1V1" (at 63.5 16.51 0)
-      (effects (font (size 1.27 1.27)))
-    )
-    (property "Footprint" "" (at 63.5 20.32 0)
-      (effects (font (size 1.27 1.27)) hide)
-    )
-    (property "Datasheet" "" (at 63.5 20.32 0)
-      (effects (font (size 1.27 1.27)) hide)
-    )
-    (pin "1")
-    (instances
-      (project "Logic_Board"
-        (path "/02d89edf-b12c-4e48-a419-0665a4b8b6d0"
-          (reference "#PWR010") (unit 1)
-        )
-      )
-      (project "T1000"
-        (path "/12aa2e34-1e28-4012-9c9f-3fbc422880b2"
-          (reference "#PWR012") (unit 1)
-        )
-      )
-      (project "Rudolph_Tracker"
-        (path "/131b2a79-e29c-42e9-9adf-d7be6c6c28ff"
-          (reference "#PWR010") (unit 1)
-        )
-      )
-      (project "SLAPS_Solar_Harvester"
-        (path "/65c91e2c-c4db-441a-a788-9bcdc306326f"
-          (reference "#PWR0107") (unit 1)
-        )
-      )
-      (project "BPP_Logger"
-        (path "/974c48bf-534e-4335-98e1-b0426c783e99"
-          (reference "#PWR06") (unit 1)
-        )
-      )
-      (project "GPS_Tracker"
-        (path "/b438986c-8622-4db9-bd4a-ee46786798d0"
-          (reference "#PWR010") (unit 1)
-        )
-      )
-      (project "Main board"
-        (path "/be354753-d7ed-4d26-938b-99a92979eaa8"
-          (reference "#PWR07") (unit 1)
-        )
-      )

Commit message: Routing actually done and made smaller????
Changed lines of the file:
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@@
+    (effects (font (size 1.27 1.27)) (justify left bottom))
+  )
+  (label "5V_R" (at 367.03 336.55 0) (fields_autoplaced)
     (effects (font (size 1.27 1.27)) (justify left bottom))
   )
   (label "SWCLK" (at 49.53 121.92 180) (fields_autoplaced)
+    (effects (font (size 1.27 1.27)) (justify right bottom))
+  )
+  (label "5V" (at 166.37 274.32 0) (fields_autoplaced)
+    (effects (font (size 1.27 1.27)) (justify left bottom))
+  )
+  (label "5V_R" (at 502.92 231.14 180) (fields_autoplaced)
     (effects (font (size 1.27 1.27)) (justify right bottom))
   )
@@
     (effects (font (size 1.27 1.27)) (justify right bottom))
   )
+  (label "5V" (at 60.96 393.7 0) (fields_autoplaced)
+    (effects (font (size 1.27 1.27)) (justify left bottom))
+  )
   (label "SWCLK_R" (at 398.78 123.19 180) (fields_autoplaced)

Commit message: Adjusted/added things
Parts:
- added J1: Conn_01x02_Socket, Connector_Molex:Molex_SL_171971-0002_1x02_P2.54mm_Vertical, symbol Connector:Conn_01x02_Socket
- added J3: Conn_01x04_Socket, Connector_Molex:Molex_SL_171971-0004_1x04_P2.54mm_Vertical, symbol Connector:Conn_01x04_Socket
- added JP1 (x2): SolderJumper_2_Open, Jumper:SolderJumper-2_P1.3mm_Open_TrianglePad1.0x1.5mm, symbol Jumper:SolderJumper_2_Open
- added R12: 10k, Resistor_SMD:R_0402_1005Metric, symbol Device:R_Small
Connections:
- net +3V3: now also JP1.2 (B), R12.1
- net +5V: now also JP1.2 (B)
- net BUSY: now also U1.36 (GPIO24); no longer U1.37 (GPIO25)
- net GND: now also J1.2 (Pin_2), J3.2 (Pin_2)
- net ~{RST}: now also U1.37 (GPIO25); no longer U1.36 (GPIO24)
- net STEP: now reaches U1.40 (GPIO28_ADC2)
- net STEP: now also J3.3 (Pin_3)
- net DIR: now reaches U1.41 (GPIO29_ADC3)
- net DIR: now also J3.4 (Pin_4)
- net PWM_ART renamed LS2
- net LS2: now also J1.1 (Pin_1), R12.2
- new net: J3.1 (Pin_1), JP1.1 (A), JP1.1 (A)
- no-connect marks 47 -> 45
Other:
- note added: "Move GPS to I2C if more pins are needed"
- note removed: "This muxing work needs to be doubled checked by someone sane"
- moved on the sheet: C1, C2, C21, J1, R12, R13, U1, U6

Commit message: Resistor size change
Parts:
- AE1: footprint Rudolph_Lib:ANT_1575AT_JOT-M -> BPPlib:ANT_1575AT_JOT-M
- C1, C10, C11, C12, C13, C14, C19, C2, C20, C21, C3, C4, C45, C46, C47, C48, C49, C5, C50, C51, C52, C53, C54, C55, C56, C6, C7, C8, C9: footprint Capacitor_SMD:C_0402_1005Metric -> Capacitor_SMD:C_0603_1608Metric
- C32, C33, C34, C38, C39, C40, C41, C42: footprint Capacitor_SMD:C_0603_1608Metric_Pad1.08x0.95mm_HandSolder -> Capacitor_SMD:C_0603_1608Metric
- L2: footprint Terminator_Lib:L_Bourns_SRP1265A -> BPPlib:L_Bourns_SRP1265A
- R1, R12, R13, R15, R16, R2, R21, R22, R3, R32, R33, R34, R35, R36, R37, R38, R39, R4, R40, R41, R42, R43, R45, R46, R47, R48, R49, R5, R50, R51, R52, R53, R54, R55, R56, R57, R58, R59, R6, R60, R61, R62, R7, R8: footprint Resistor_SMD:R_0402_1005Metric -> Resistor_SMD:R_0603_1608Metric
- TP1, TP2: footprint TestPoint:TestPoint_Pad_D1.0mm -> TestPoint:TestPoint_Keystone_5000-5004_Miniature
Other:
- note added: "Shipman is currently testing :("
- note removed: "Shipman is currently testing"

Commit message: fixed the drc things that are problems
Parts:
- added TP10, TP5, TP6, TP7, TP8, TP9: TestPoint, TestPoint:TestPoint_Keystone_5000-5004_Miniature, symbol Connector:TestPoint
- U1: footprint Package_LGA:LGA-14_3x2.5mm_P0.5mm_LayoutBorder3x4y -> BPPlib:BMI270_BOS-L
Connections:
- net +3V3: now also TP5.1, TP8.1
- net +5V: now also TP6.1, TP7.1
- net SCL: now also TP10.1
- net SDA: now also TP9.1

Commit message: minor changes
Parts:
- J1, JP1, JP2: now left out of the parts list
Other:
- title: (none) -> Bobot-2
Changed lines of the file:
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@@
 	(generator_version "8.0")
 	(paper "C")
+	(title_block
+		(title "Bobot-2")
+		(date "2024-03-18")
+	)
 	(junction
 		(at 121.92 361.95)
@@
 		(unit 1)
 		(exclude_from_sim no)
-		(in_bom yes)
+		(in_bom no)
 		(on_board yes)
 		(dnp no)
@@
 		(unit 1)
 		(exclude_from_sim no)
-		(in_bom yes)
+		(in_bom no)
 		(on_board yes)
 		(dnp no)
@@
 		(unit 1)
 		(exclude_from_sim no)
-		(in_bom yes)
+		(in_bom no)
 		(on_board yes)
 		(dnp no)
@@
 		(unit 1)
 		(exclude_from_sim no)
-		(in_bom yes)
+		(in_bom no)
 		(on_board yes)
 		(dnp no)

Commit message: Update changes hopefully good
Parts:
- removed C32, C33: 220nF, Capacitor_SMD:C_0603_1608Metric, symbol Device:C_Small
- removed C34: 4.7uF, Capacitor_SMD:C_0603_1608Metric, symbol Device:C_Small
- removed C38: 22nF, Capacitor_SMD:C_0603_1608Metric, symbol Device:C_Small
- removed C39, C40: 22uF, Capacitor_SMD:C_0603_1608Metric, symbol Device:C_Small
- removed C41: 680p, Capacitor_SMD:C_0603_1608Metric, symbol Device:C_Small
- removed C42: 10uF, Capacitor_SMD:C_0603_1608Metric, symbol Device:C_Small
- removed J4: Nichrome, Connector_PinHeader_2.54mm:PinHeader_1x02_P2.54mm_Vertical, symbol Connector:Conn_01x02_Socket
- removed JP1, JP2: SolderJumper_2_Open, Jumper:SolderJumper-2_P1.3mm_Open_TrianglePad1.0x1.5mm, symbol Jumper:SolderJumper_2_Open
- removed L2: 3.3uH, BPPlib:L_Bourns_SRP1265A, symbol Device:L
- removed R23: 81.1k, Resistor_SMD:R_0603_1608Metric_Pad0.98x0.95mm_HandSolder, symbol Device:R_Small
- removed R24: 75k, Resistor_SMD:R_0603_1608Metric_Pad0.98x0.95mm_HandSolder, symbol Device:R_Small
- removed R25: 5m, Resistor_SMD:R_0603_1608Metric_Pad0.98x0.95mm_HandSolder, symbol Device:R_Small
- removed R26, R27: 154k, Resistor_SMD:R_0603_1608Metric_Pad0.98x0.95mm_HandSolder, symbol Device:R_Small
- removed R28: 56.2k, Resistor_SMD:R_0603_1608Metric_Pad0.98x0.95mm_HandSolder, symbol Device:R_Small
- removed U1: LT3120JV-PBF, BPPlib:LQFN28_Rev0_ADI, symbol Terminator_Lib:LT3120JV-PBF
- removed Y1 (x2): 445I23D12M00000, Crystal:Crystal_SMD_5032-2Pin_5.0x3.2mm, symbol Device:Crystal_Small
- added 0.3_Ohm_Resistor1: 03, Package_TO_SOT_SMD:TO-263-2, symbol Device:R
- added C58: 100nF, Capacitor_SMD:C_0603_1608Metric, symbol Device:C_Small
- added C59: 1uF, Capacitor_SMD:C_0603_1608Metric, symbol Device:C_Small
- added J11: Conn_01x02_Pin, Connector_Molex:Molex_SL_171971-0002_1x02_P2.54mm_Vertical, symbol Connector:Conn_01x02_Pin
- added J17: Conn_01x04_Pin, Connector_Molex:Molex_SL_171971-0004_1x04_P2.54mm_Vertical, symbol Connector:Conn_01x04_Pin
- added J18: Conn_01x03_Socket, Connector_Molex:Molex_SL_171971-0003_1x03_P2.54mm_Vertical, symbol Connector:Conn_01x03_Socket
- added JP2: SolderJumper_2_Bridged, Jumper:SolderJumper-2_P1.3mm_Bridged_Pad1.0x1.5mm, symbol Jumper:SolderJumper_2_Bridged
- added LM1084-ADJ1: LM1084-ADJ, Package_TO_SOT_SMD:TO-263-3_TabPin2, symbol Regulator_Linear:LM1084-ADJ
- added MOSFET2: IRF540N, Package_TO_SOT_SMD:TO-252-2, symbol Transistor_FET:IRF540N
- added Y1, Y2: 12MHz, Crystal:Crystal_SMD_2520-4Pin_2.5x2.0mm, symbol Device:Crystal_GND24_Small
- C1, C2: value 22pF -> 10pF
- J4: footprint Connector_Coaxial:U.FL_Molex_MCRF_73412-0110_Vertical -> Connector_Coaxial:SMA_Amphenol_132289_EdgeMount
Connections:
- net +3V3: now also C58.1, C59.1; no longer C10.1, C11.1, C12.1, C13.1, C14.1, C15.1, C49.1, C6.1, C7.1, C8.1, C9.1, J1.1 (Pin_1), R2.1, R38.1, R8.1, R9.1, TP8.1, U1.1 (IOVDD), U1.10 (IOVDD), U1.22 (IOVDD), U1.33 (IOVDD), U1.42 (IOVDD), U1.43 (ADC_AVDD), U1.44 (VREG_IN), U1.48 (USB_VDD), U1.49 (IOVDD), U12.1 (VOUT), U12.2 (SENSE), U2.8 (VCC)
- net +5V: now also J18.1 (Pin_1); no longer C50.1, J4.1 (Pin_1), R39.1, TP7.1, U13.1 (VOUT), U13.2 (SENSE)
- net +BATT: now also J16.1 (Pin_1), R55.2, R58.2, U15.7 (IN1), LM1084-ADJ1.3 (VI)
- net CUT: now also J17.2 (Pin_2), JP2.1 (A)
- net GND: now also 0.3_Ohm_Resistor1.3 (Gnd), C58.2, C59.2, J17.1 (Pin_1), J18.3 (Pin_3), MOSFET2.3 (S), Y1.2, Y1.4, Y2.2, Y2.4
- net PWM_MC: now also J18.2 (Pin_2)
- net at C2.2, R1.1: now also Y2.1
- net at C1.2, U1.20 (XIN): now also Y2.3
- net at C1.2, U1.20 (XIN): now also Y1.3
- net at C2.2, R1.1: now also Y1.1
- new net: 0.3_Ohm_Resistor1.1, J11.2 (Pin_2), LM1084-ADJ1.1 (ADJ)
- new net: 0.3_Ohm_Resistor1.2, LM1084-ADJ1.2 (VO)
- new net: JP2.2 (B), MOSFET2.1 (G)
- new net: J11.1 (Pin_1), MOSFET2.2 (D)
- new net +3V3_R: C10.1, C11.1, C12.1, C13.1, C14.1, C15.1, C49.1, C6.1, C7.1, C8.1, C9.1, J1.1 (Pin_1), J17.3 (Pin_3), R2.1, R38.1, R8.1, R9.1, TP8.1, U1.1 (IOVDD), U1.10 (IOVDD), U1.22 (IOVDD), U1.33 (IOVDD), U1.42 (IOVDD), U1.43 (ADC_AVDD), U1.44 (VREG_IN), U1.48 (USB_VDD), U1.49 (IOVDD), U12.1 (VOUT), U12.2 (SENSE), U2.8 (VCC)
- new net +5V_R: C50.1, J17.4 (Pin_4), J4.1 (Pin_1), R39.1, TP7.1, U13.1 (VOUT), U13.2 (SENSE)
- no-connect marks 45 -> 44
Other:
- note added: "Motor Controller"
- note added: "PICO(Peripheral in controller out) POCI(Peripheral out controller in)"
- note removed: "Shipman is currently testing :("
- company: (none) -> UMD Balloon Payload Program
- moved on the sheet: C55, C56, J1, R47, R48, R49, R54, R56, R57
