File: Hardware/Tim/Main board/Main board.kicad_sch (KiCad schematic)
At the start: 171 parts, among them J1 Conn_01x02_Socket, J1 SOICbite, J11 Conn_01x02_Pin, J14 Conn_01x02_Pin, J16 Conn_01x02_Pin, J17 Conn_01x04_Pin, J18 Conn_01x03_Socket, J2 USB_C_Receptacle_USB2.0, J3 Conn_01x04_Socket, J4 Conn_01x03_Socket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

Commit message: Updated things
Parts:
- added C37, C39, C41, C43: 1uF, Capacitor_SMD:C_0603_1608Metric, symbol Device:C
- added C38, C40, C42, C44: 100nF, Capacitor_SMD:C_0603_1608Metric, symbol Device:C
Connections:
- net +BATT: now also C43.1, C44.1
- net GND: now also C37.2, C38.2, C39.2, C40.2, C41.2, C42.2, C43.2, C44.2
- net VBUS: now also C37.1, C38.1
- net VCC: now also C41.1, C42.1
- net at J14.1 (Pin_1), R45.2, R46.2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: now also C39.1, C40.1
Other:
- moved on the sheet: J14, J16

Commit message: Double checking everything is pushed
Parts:
- added J19, J20: Micro_SD_Card, BPPlib:JAE_ST1W008S4ER1500, symbol Connector:Micro_SD_Card
Connections:
- net +3V3: now also J19.4 (VDD)
- net +3V3_R: now also J20.4 (VDD)
- net EXTINT: no longer U1.38 (GPIO26_ADC0)
- net GND: now also J19.6 (VSS), J19.9 (SHIELD), J20.6 (VSS), J20.9 (SHIELD)
- net SPI0_PICO: now also J19.3 (CMD)
- net SPI0_POCI: now also J19.7 (DAT0)
- net SPI0_SCK: now also J19.5 (CLK)
- net TXEN: now also U1.38 (GPIO26_ADC0); no longer U1.32 (GPIO21)
- net SPI0_POCI_R: now reaches U1.15 (GPIO12)
- net SPI0_POCI_R: now also J20.7 (DAT0)
- net SPI0_CS_SD_R: now reaches U1.16 (GPIO13)
- net SPI0_CS_SD_R: now also J20.2 (DAT3/CD)
- net SPI0_SCK_R: now reaches U1.17 (GPIO14)
- net SPI0_SCK_R: now also J20.5 (CLK)
- net SPI0_PICO_R: now reaches U1.18 (GPIO15)
- net SPI0_PICO_R: now also J20.3 (CMD)
- new net SPI0_CS_SD: J19.2 (DAT3/CD), U1.32 (GPIO21)
Other:
- moved on the sheet: B2, C13, R7, R8, U2
