File: Hardware/Tim/main_board2.0/winderboard_2.0/winderboard_2.0.kicad_sch (KiCad schematic)
At the start: 21 parts, among them J1 Conn_01x03_Socket, J10 Conn_01x04_Socket, J11 Conn_01x06_Socket, J2 Conn_01x03_Socket, J3 Conn_01x03_Socket, J4 Conn_01x03_Socket, J5 Conn_01x05_Socket, J6 Conn_01x05_Socket, J7 Conn_01x05_Socket, J8 Conn_01x02_Socket, J9 Conn_01x02_Socket, U1 DEV-16771, U2 MS5607-02BA, U3 MAX-M10S, U4 TMP100

Commit message: latest changes
Parts:
- R1, R2: value R_Small -> 4.7k
Connections:
- net +3.3V: now reaches R2.1
- net +3.3V: now also J1.2 (Pin_2), J2.2 (Pin_2), R1.1
- net at R2.2: now also J2.1 (Pin_1)
- net at R1.2: now also J1.1 (Pin_1)
- net GND: now reaches J1.3 (Pin_3)
- net GND: now also J2.3 (Pin_3)
Other:
- moved on the sheet: J1, R1, R2

Commit message: latest board
Parts:
- removed J3, J4: Conn_01x03_Socket, symbol Connector:Conn_01x03_Socket
- removed J7: Conn_01x05_Socket, symbol Connector:Conn_01x05_Socket
- added A1: Pololu_Breakout_A4988, Module:Pololu_Breakout-16_15.2x20.3mm, symbol Driver_Motor:Pololu_Breakout_A4988
- added BT2: BAT-HLD-001, BAT-HLD-001:BAT_BAT-HLD-001, symbol BAT-HLD-001:BAT-HLD-001
- added BT3: motor_batt, symbol Device:Battery_Cell
- added C4: 100nF, symbol Device:C_Small
- added C5: C_Small, symbol Device:C_Small
- added J12: Conn_01x04_Socket, symbol Connector:Conn_01x04_Socket
- added J3, J4: Conn_01x02_Socket, symbol Connector:Conn_01x02_Socket
- added J7: Conn_01x03_Socket, symbol Connector:Conn_01x03_Socket
- added M1: Stepper_Motor_bipolar, symbol Motor:Stepper_Motor_bipolar
- added Q1, Q2: NMOS, Package_TO_SOT_SMD:SOT-23-3, symbol Simulation_SPICE:NMOS
- added R3, R4: 10k, symbol Device:R_Small
- added R5, R6: R_Small, symbol Device:R_Small
- BT1: value Battery_Cell -> GPS_Batt
- C1: value C_Small -> 1uF
- C2: value C_Small -> 100nF
- C3: value C_Small -> 10uF
Connections:
- net +3.3V: now also C1.1, C2.2, U1.10 (CS1), U1.9 (OUT1C), U2.1 (VDD), U2.2 (PS), U3.7 (VCC_IO), U3.8 (VCC), U4.4 (V+), C4.1, R3.1, R4.1
- net GND: now also BT1.2 (-), C1.2, C2.1, C3.2, J10.4 (Pin_4), J11.3 (Pin_3), J5.5 (Pin_5), J6.5 (Pin_5), U1.GND1 (GND), U1.GND2 (GND), U1.GND3 (GND), U1.GND4 (GND), U1.GND5 (GND), U2.3 (GND), U2.4 (CSB), U2.5 (CSB), U3.1 (GND), U3.10 (GND), U3.12 (GND), U4.2 (GND), U4.3 (ADD1), U4.5 (ADD0), A1.1 (GND), A1.7 (GND), BT2.N1, BT3.2 (-), C4.2, C5.2, J12.2 (Pin_2), J3.2 (Pin_2), J4.2 (Pin_2), J7.3 (Pin_3), Q1.3 (S), Q2.3 (S)
- net at C3.1: now also BT1.1 (+), U3.6 (V_BCKP)
- net xbee_RX: now reaches J10.1 (Pin_1)
- net xbee_RX: now also U1.8 (TX2)
- net xbee_TX: now reaches J10.2 (Pin_2)
- net xbee_TX: now also U1.7 (RX2)
- net +5V: now reaches J10.3 (Pin_3)
- net +5V: now also J11.1 (Pin_1), J5.2 (Pin_2), J6.2 (Pin_2), J8.1 (Pin_1), J9.1 (Pin_1), A1.2 (VDD), J12.1 (Pin_1)
- net IR_SDA: now reaches U2.7 (SDI/SDA)
- net IR_SDA: now also U1.18 (A4), U4.6 (SDA), J12.4 (Pin_4), R4.2
- net IR_SCL: now reaches U2.8 (SCLK)
- net IR_SCL: now also U1.19 (A5), U4.1 (SCL), J12.3 (Pin_3), R3.2
- net encoder_B2: now reaches J6.1 (Pin_1)
- net encoder_A2: now reaches J6.3 (Pin_3)
- net encoder_X2: now reaches J6.4 (Pin_4)
- net IMU_SDA: now reaches J11.5 (Pin_5)
- net IMU_SDA: now also U1.17 (A3)
- net IMU_SCL: now reaches J11.6 (Pin_6)
- net IMU_SCL: now also U1.16 (A2)
- net at J8.2 (Pin_2): now also Q1.1 (D)
- net encoder_B1: now reaches J5.1 (Pin_1)
- net encoder_A1: now reaches J5.3 (Pin_3)
- net encoder_X1: now reaches J5.4 (Pin_4)
- net at U3.2 (TXD): now also R6.2
- net at U3.3 (RXD): now also R5.2
- net GPS_TX: now reaches U1.0 (RX1)
- net GPS_TX: now also R6.1
- net GPS_RX: now reaches U1.1 (TX1)
- net GPS_RX: now also R5.1
- net stepper_step: now reaches U1.2 (OUT2)
- net stepper_step: now also A1.15 (STEP)
- net stepper_dir: now reaches U1.3 (LRCLK2)
- net stepper_dir: now also A1.16 (DIR)
- net heater1: now reaches U1.31 (CTX3)
- net heater1: now also Q1.2 (G)
- net heater2: now reaches U1.32 (OUT1B)
- net heater2: now also Q2.2 (G)
- net BLDC_PWM: now reaches U1.33 (MCLK2)
- net BLDC_PWM: now also J7.1 (Pin_1)
- net stepper_MS1: now reaches U1.4 (BCLK2)
- net stepper_MS1: now also A1.10 (MS1)
- net limitswitch1: now reaches U1.40 (A16)
- net limitswitch1: now also J4.1 (Pin_1)
- net limitswitch2: now reaches U1.41 (A17)
- net limitswitch2: now also J3.1 (Pin_1)
- net stepper_MS2: now reaches U1.5 (IN2)
- net stepper_MS2: now also A1.11 (MS2)
- net stepper_MS3: now reaches U1.6 (OUT1D)
- net stepper_MS3: now also A1.12 (MS3)
- net RTC_Batt: now reaches U1.VBAT
- net RTC_Batt: now also BT2.P1, BT2.P2
- net +5VD: now reaches U1.VIN
- net +5VD: now also J7.2 (Pin_2)
- net at J9.2 (Pin_2): now also Q2.1 (D)
- new net: A1.4 (1A), M1.1
- new net: A1.3 (1B), M1.2 (-)
- new net: A1.5 (2A), M1.3
- new net: A1.6 (2B), M1.4
- new net +BATT: A1.8 (VMOT), BT3.1 (+), C5.1
- no-connect marks 0 -> 4
Other:
- moved on the sheet: BT1, C1, C2, C3, J1, J2, J5, J6, J9, R1, R2, U1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

Commit message: finished wiring
Parts:
- added C10: 10uF, Capacitor_SMD:C_0603_1608Metric_Pad1.08x0.95mm_HandSolder, symbol Device:C_Small
- added C6, C7: 0.1uF, symbol Device:C_Small
- added C8: 3.3nF, Capacitor_SMD:C_0603_1608Metric_Pad1.08x0.95mm_HandSolder, symbol Device:C_Small
- added C9: 0.1uF, Capacitor_SMD:C_0603_1608Metric_Pad1.08x0.95mm_HandSolder, symbol Device:C_Small
- added J13: Conn_01x02_Socket, symbol Connector:Conn_01x02_Socket
- added L1: 1uH, Inductor_SMD:L_Coilcraft_XxL4040, symbol Device:L_Small
- added M2: Motor_Servo, symbol Motor:Motor_Servo
- added Q3: DMN6040SK3-13, Package_TO_SOT_SMD:TO-252-2, symbol Transistor_FET:QM6015D
- added R7, R8: 4.7k, Resistor_SMD:R_0603_1608Metric_Pad0.98x0.95mm_HandSolder, symbol Device:R_Small
- added R9: R_Small, Resistor_SMD:R_0603_1608Metric_Pad0.98x0.95mm_HandSolder, symbol Device:R_Small
- added RV1: R_Potentiometer, symbol Device:R_Potentiometer
- added TP1: TestPoint, symbol Connector:TestPoint
- added U5: LM1084-ADJ, symbol Regulator_Linear:LM1084-ADJ
- added U6: 0.3 Ohm Resistor, Package_TO_SOT_SMD:TO-263-2, symbol Regulator_Linear:NVC8674DS50
- added U7: INA260, Package_SO:TSSOP-16_4.4x5mm_P0.65mm, symbol Sensor:INA260
- added U8: TPS62133, Package_DFN_QFN:VQFN-16-1EP_3x3mm_P0.5mm_EP1.68x1.68mm_ThermalVias, symbol Regulator_Switching:TPS62133
- C1, C2, C3, C4: footprint (none) -> Capacitor_SMD:C_0603_1608Metric_Pad1.08x0.95mm_HandSolder
- C5: value C_Small -> 100uF; footprint (none) -> Capacitor_SMD:C_0603_1608Metric_Pad1.08x0.95mm_HandSolder
- R1, R2, R3, R4, R5, R6: footprint (none) -> Resistor_SMD:R_0603_1608Metric_Pad0.98x0.95mm_HandSolder
Connections:
- net +5V: now also U1.5V, C6.1, M2.2 (+), RV1.1, U7.10 (VS)
- net +5VD: now also L1.2, R9.1, U8.14 (VOS)
- net +BATT: now also C10.1, C7.2, C9.1, U5.3 (VI), U7.1 (IN+), U7.12 (VBUS), U7.2 (IN+), U7.3 (IN+), U8.10 (VIN), U8.11 (VIN), U8.12 (VIN), U8.13 (EN)
- net BLDC_PWM: now also U1.23 (A9); no longer U1.33 (MCLK2)
- net GND: now also C10.2, C6.2, C7.1, C8.2, C9.2, M2.3 (-), Q3.3 (S), RV1.3, U6.2 (GND), U7.11 (GND), U7.4 (A1), U7.5 (A0), U7.6 (GND), U8.15 (GND), U8.16 (GND), U8.17 (GND), U8.5 (FB), U8.6 (GND), U8.7 (FSW), U8.8 (DEF)
- net encoder_A1: now also U1.33 (MCLK2)
- net encoder_A2: now also U1.36 (CS2)
- net encoder_B1: now also U1.34 (RX8)
- net encoder_B2: now also U1.37 (CS3)
- net encoder_X1: now also U1.35 (TX8)
- net encoder_X2: now also U1.38 (A14)
- net pot_data: now reaches U1.14 (A0)
- net pot_data: now also RV1.2
- net cutservo_PWM: now reaches U1.22 (A8)
- net cutservo_PWM: now also M2.1 (PWM)
- net power_SCL: now reaches U1.24 (A10)
- net power_SCL: now also R7.2
- net power_SDA: now reaches U1.25 (A11)
- net power_SDA: now also R8.1
- net cutdown: now reaches U1.30 (CRX3)
- net cutdown: now also Q3.1 (G)
- new net: R8.2, U7.8 (SDA)
- new net: R7.1, U7.9 (SCL)
- new net: L1.1, U8.1 (SW), U8.2 (SW), U8.3 (SW)
- new net: R9.2, TP1.1, U8.4 (PG)
- new net: C8.1, U8.9 (SS/TR)
- new net: U5.2 (VO), U6.1 (IN)
- new net: J13.1 (Pin_1), U5.1 (ADJ), U6.3 (OUT)
- new net: J13.2 (Pin_2), Q3.2 (D)
- new net -BATT: U7.14 (IN-), U7.15 (IN-), U7.16 (IN-)
Other:
- moved on the sheet: BT3, J1, J12, J2, J3, J4, R1, R2

Commit message: actually done with schematic
Parts:
- added J14: Conn_01x10_Pin, Connector_PinHeader_2.54mm:PinHeader_1x10_P2.54mm_Vertical, symbol Connector:Conn_01x10_Pin
- added J15: Conn_01x04_Pin, Connector_PinHeader_2.54mm:PinHeader_1x04_P2.54mm_Vertical, symbol Connector:Conn_01x04_Pin
- added R10: 4.7k, symbol Device:R_Small
- BT1: footprint (none) -> ML414H_IV01E:SEIKO_ML414H_IV01E
- BT3: footprint (none) -> Connector_AMASS:AMASS_XT30PW-M_1x02_P2.50mm_Horizontal
- C6, C7: footprint (none) -> Capacitor_SMD:C_0603_1608Metric_Pad1.08x0.95mm_HandSolder
- J1, J2, M2: footprint (none) -> Connector_JST:JST_EH_B3B-EH-A_1x03_P2.50mm_Vertical
- J12, M1: footprint (none) -> Connector_JST:JST_EH_B4B-EH-A_1x04_P2.50mm_Vertical
- J3, J4, J8, J9: footprint (none) -> Connector_JST:JST_XH_B2B-XH-A_1x02_P2.50mm_Vertical
- J5, J6: footprint (none) -> Connector_JST:JST_XH_B5B-XH-AM_1x05_P2.50mm_Vertical
- RV1: footprint (none) -> Connector_JST:JST_XH_B3B-XH-A_1x03_P2.50mm_Vertical
- U5: footprint (none) -> Package_TO_SOT_SMD:TO-263-3_TabPin2
Connections:
- net +3.3V: now also U1.3.3V_1 (3.3V), U1.3.3V_2 (3.3V), U1.3.3V_3 (3.3V), U1.39 (A15); no longer U1.10 (CS1)
- net +5V: now also J12.2 (Pin_2), J8.2 (Pin_2), J9.2 (Pin_2), L1.2, R9.1, RV1.3, U1.VIN, U8.14 (VOS); no longer J12.1 (Pin_1), J8.1 (Pin_1), J9.1 (Pin_1), RV1.1
- net GND: now also J12.1 (Pin_1), J3.1 (Pin_1), J4.1 (Pin_1), J5.1 (Pin_1), J6.1 (Pin_1), RV1.1, R10.2; no longer J12.2 (Pin_2), J3.2 (Pin_2), J4.2 (Pin_2), J5.5 (Pin_5), J6.5 (Pin_5), RV1.3
- net encoder_B1: now also J5.5 (Pin_5); no longer J5.1 (Pin_1)
- net encoder_B2: now also J6.5 (Pin_5); no longer J6.1 (Pin_1)
- net limitswitch1: now also J4.2 (Pin_2); no longer J4.1 (Pin_1)
- net limitswitch2: now also J3.2 (Pin_2); no longer J3.1 (Pin_1)
- net stepper_sleep: now reaches A1.14 (~{SLEEP})
- net stepper_sleep: now also U1.15 (A1), R10.1
- net at Q1.1 (D): now also J8.1 (Pin_1); no longer J8.2 (Pin_2)
- net at Q2.1 (D): now also J9.1 (Pin_1); no longer J9.2 (Pin_2)
- net 11: now reaches U1.11 (MOSI)
- net 11: now also J14.2 (Pin_2)
- net 12: now reaches U1.12 (MISO)
- net 12: now also J14.3 (Pin_3)
- net 13: now reaches U1.13 (SCK)
- net 13: now also J14.4 (Pin_4)
- net 20: now reaches U1.20 (A6)
- net 20: now also J14.5 (Pin_5)
- net 21: now reaches U1.21 (A7)
- net 21: now also J14.6 (Pin_6)
- net 26: now reaches U1.26 (A12)
- net 26: now also J14.7 (Pin_7)
- net 27: now reaches U1.27 (A13)
- net 27: now also J14.8 (Pin_8)
- net 28: now reaches U1.28 (RX7)
- net 28: now also J14.9 (Pin_9)
- net 29: now reaches U1.29 (TX7)
- net 29: now also J14.10 (Pin_10)
- removed net +5VD: J7.2 (Pin_2), L1.2, R9.1, U1.VIN, U8.14 (VOS)
- net IMU_SCL renamed I2C_SCL2
- net I2C_SCL2: now also J15.3 (Pin_3)
- net IMU_SDA renamed I2C_SDA2
- net I2C_SDA2: now also J15.4 (Pin_4)
- net power_SCL renamed I2C_SCL1
- net I2C_SCL1: now also J15.2 (Pin_2)
- net power_SDA renamed I2C_SDA1
- net I2C_SDA1: now also J15.1 (Pin_1)
- new net 10: J14.1 (Pin_1), U1.10 (CS1)
- no-connect marks 4 -> 16
Other:
- moved on the sheet: BT3, J3, J4, J8, J9, Q2, RV1

Commit message: started working on layout
Parts:
- J11: footprint (none) -> BNO055:BNO055
- J13: footprint (none) -> Connector_PinHeader_2.54mm:PinHeader_1x02_P2.54mm_Vertical
- J7: footprint (none) -> Connector_JST:JST_EH_B3B-EH-A_1x03_P2.50mm_Vertical
- R10: footprint (none) -> Resistor_SMD:R_0603_1608Metric_Pad0.98x0.95mm_HandSolder
- TP1: footprint (none) -> TestPoint:TestPoint_Loop_D2.54mm_Drill1.5mm_Beaded
Connections:
- net I2C_SCL2: now also J11.5 (Pin_5); no longer J11.6 (Pin_6)
- net I2C_SDA2: now also J11.4 (Pin_4); no longer J11.5 (Pin_5)
- no-connect marks 16 -> 18
Changed lines of the file:
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@@
 	)
 	(no_connect
-		(at 179.07 245.11)
-	)
-	(no_connect
 		(at 106.68 54.61)
 	)
@@
 	)
 	(no_connect
+		(at 179.07 250.19)
+	)
+	(no_connect
 		(at 66.04 44.45)
 	)
@@
 	)
 	(no_connect
+		(at 57.15 191.77)
+	)
+	(no_connect
 		(at 106.68 46.99)
 	)
@@
 		(at 106.68 29.21)
 	)
+	(no_connect
+		(at 57.15 189.23)
+	)
 	(wire
 		(pts
@@
 		)
 	)
-	(global_label "IMU_SCL"
-		(shape input)
-		(at 179.07 250.19 180)
-		(fields_autoplaced yes)
-		(effects
-			(font
-				(size 1.27 1.27)
-			)
-			(justify right)
-		)
-		(property "Intersheetrefs" "${INTERSHEET_REFS}"
-			(at 168.2229 250.19 0)
-			(effects
-				(font
-					(size 1.27 1.27)
-				)
-				(justify right)
-				(hide yes)
-			)
-		)
-	)
 	(global_label "I2C_SCL2"
 		(shape input)
@@
 		)
 	)
+	(global_label "IMU_SDA"
+		(shape input)
+		(at 179.07 245.11 180)
+		(fields_autoplaced yes)
+		(effects
+			(font
+				(size 1.27 1.27)
+			)
+			(justify right)
+		)
+		(property "Intersheetrefs" "${INTERSHEET_REFS}"
+			(at 168.1624 245.11 0)
+			(effects
+				(font
+					(size 1.27 1.27)
+				)
+				(justify right)
+				(hide yes)
+			)
+		)
+	)
 	(global_label "GPS_RX"
 		(shape input)
@@
 		)
 	)
+	(global_label "IMU_SCL"
+		(shape input)
+		(at 179.07 247.65 180)
+		(fields_autoplaced yes)
+		(effects
+			(font
+				(size 1.27 1.27)
+			)
+			(justify right)
+		)
+		(property "Intersheetrefs" "${INTERSHEET_REFS}"
+			(at 168.2229 247.65 0)
+			(effects
+				(font
+					(size 1.27 1.27)
+				)
+				(justify right)
+				(hide yes)
+			)
+		)
+	)
 	(global_label "stepper_MS2"
 		(shape input)
@@
 		)
 	)
-	(global_label "IMU_SDA"
-		(shape input)
-		(at 179.07 247.65 180)
-		(fields_autoplaced yes)
-		(effects
-			(font
-				(size 1.27 1.27)
-			)
-			(justify right)
-		)
-		(property "Intersheetrefs" "${INTERSHEET_REFS}"
-			(at 168.1624 247.65 0)
-			(effects
-				(font
-					(size 1.27 1.27)
-				)
-				(justify right)
-				(hide yes)
-			)
-		)
-	)
 	(global_label "RTC_Batt"
 		(shape input)
@@
 			)
 		)
-		(property "Footprint" ""
+		(property "Footprint" "Resistor_SMD:R_0603_1608Metric_Pad0.98x0.95mm_HandSolder"
 			(at 278.13 110.49 0)
 			(effects
@@
 			)
 		)
-		(property "Footprint" ""
+		(property "Footprint" "Connector_JST:JST_EH_B3B-EH-A_1x03_P2.50mm_Vertical"
 			(at 172.72 147.32 0)
 			(effects
@@
 			)
 		)
-		(property "Footprint" ""
+		(property "Footprint" "TestPoint:TestPoint_Loop_D2.54mm_Drill1.5mm_Beaded"
 			(at 83.82 251.46 0)
 			(effects
@@
 			)
 		)
-		(property "Footprint" ""
+		(property "Footprint" "BNO055:BNO055"
 			(at 184.15 242.57 0)
 			(effects
@@
 			)
 		)
-		(property "Footprint" ""
+		(property "Footprint" "Connector_PinHeader_2.54mm:PinHeader_1x02_P2.54mm_Vertical"
 			(at 379.73 50.8 0)
 			(effects

Commit message: First draft of final
Parts:
- removed C2: 100nF, Capacitor_SMD:C_0603_1608Metric_Pad1.08x0.95mm_HandSolder, symbol Device:C_Small
- removed C6, C7: 0.1uF, Capacitor_SMD:C_0603_1608Metric_Pad1.08x0.95mm_HandSolder, symbol Device:C_Small
- removed J14: Conn_01x10_Pin, Connector_PinHeader_2.54mm:PinHeader_1x10_P2.54mm_Vertical, symbol Connector:Conn_01x10_Pin
- removed R7, R8: 4.7k, Resistor_SMD:R_0603_1608Metric_Pad0.98x0.95mm_HandSolder, symbol Device:R_Small
- removed U4: TMP100, Package_TO_SOT_SMD:SOT-23-6, symbol Sensor_Temperature:TMP100
- removed U7: INA260, Package_SO:TSSOP-16_4.4x5mm_P0.65mm, symbol Sensor:INA260
- added C11: 22uF, Capacitor_SMD:C_0603_1608Metric_Pad1.08x0.95mm_HandSolder, symbol Device:C_Small
- added D1: D_Schottky, Diode_SMD:D_SOD-123F, symbol Device:D_Schottky
- added J14: Conn_Coaxial, Connector_Coaxial:U.FL_Molex_MCRF_73412-0110_Vertical, symbol Connector:Conn_Coaxial
- added J16: INA260, Connector_JST:JST_XH_B4B-XH-A_1x04_P2.50mm_Vertical, symbol Connector:Conn_01x04_Socket
- added J17: Conn_01x04_Socket, Connector_JST:JST_XH_B4B-XH-A_1x04_P2.50mm_Vertical, symbol Connector:Conn_01x04_Socket
- added J18: Conn_01x08_Pin, Connector_PinHeader_2.54mm:PinHeader_1x08_P2.54mm_Vertical, symbol Connector:Conn_01x08_Pin
- added J19: Conn_01x01_Pin, MountingHole:MountingHole_3.2mm_M3_DIN965_Pad, symbol Connector:Conn_01x01_Pin
- added R11: 3.3k, Resistor_SMD:R_0603_1608Metric_Pad0.98x0.95mm_HandSolder, symbol Device:R_Small
- BT2: value BAT-HLD-001 -> RTC Battery
- J1: value Conn_01x03_Socket -> Temp Probe 1; footprint Connector_JST:JST_EH_B3B-EH-A_1x03_P2.50mm_Vertical -> Connector_JST:JST_XH_B3B-XH-A_1x03_P2.50mm_Vertical
- J10: value Conn_01x04_Socket -> XBee Explorer
- J11: value Conn_01x06_Socket -> BNO055
- J12: value Conn_01x04_Socket -> IR Temp Sensor; footprint Connector_JST:JST_EH_B4B-EH-A_1x04_P2.50mm_Vertical -> Connector_JST:JST_XH_B4B-XH-A_1x04_P2.50mm_Vertical
- J15: value Conn_01x04_Pin -> I2C Pinout
- J2: value Conn_01x03_Socket -> Temp Probe 2; footprint Connector_JST:JST_EH_B3B-EH-A_1x03_P2.50mm_Vertical -> Connector_JST:JST_XH_B3B-XH-A_1x03_P2.50mm_Vertical
- J3: value Conn_01x02_Socket -> Limit Switch 2
- J4: value Conn_01x02_Socket -> Limit Switch 1
- J5: value Conn_01x05_Socket -> Encoder 1; footprint Connector_JST:JST_XH_B5B-XH-AM_1x05_P2.50mm_Vertical -> Connector_JST:JST_XH_B5B-XH-A_1x05_P2.50mm_Vertical
- J6: value Conn_01x05_Socket -> Encoder 2; footprint Connector_JST:JST_XH_B5B-XH-AM_1x05_P2.50mm_Vertical -> Connector_JST:JST_XH_B5B-XH-A_1x05_P2.50mm_Vertical
- J7: value Conn_01x03_Socket -> ESC; footprint Connector_JST:JST_EH_B3B-EH-A_1x03_P2.50mm_Vertical -> Connector_JST:JST_XH_B3B-XH-A_1x03_P2.50mm_Vertical
- J8: value Conn_01x02_Socket -> Heater 1
- J9: value Conn_01x02_Socket -> Heater 2
- M1: footprint Connector_JST:JST_EH_B4B-EH-A_1x04_P2.50mm_Vertical -> Connector_JST:JST_XH_B4B-XH-A_1x04_P2.50mm_Vertical
- M2: footprint Connector_JST:JST_EH_B3B-EH-A_1x03_P2.50mm_Vertical -> Connector_JST:JST_XH_B3B-XH-A_1x03_P2.50mm_Vertical
- R5, R6: value R_Small -> ??
Connections:
- net 26 is gone; now on net EXTINT: U1.26 (A12)
- net 27 is gone; now on net TIMEPULSE: U1.27 (A13)
- net +3.3V: now also J1.3 (Pin_3), J2.3 (Pin_3), R1.2, R2.2, D1.2 (A); no longer J1.2 (Pin_2), J2.2 (Pin_2), R1.1, R2.1, U1.39 (A15), U1.9 (OUT1C)
- net +5V: now also C11.1, J16.4 (Pin_4), J18.2 (Pin_2)
- net +BATT: now also J17.4 (Pin_4)
- net 10: now also J18.3 (Pin_3)
- net 11: now also J18.4 (Pin_4)
- net 12: now also J18.5 (Pin_5)
- net 13: now also J18.6 (Pin_6)
- net 28: now also J18.7 (Pin_7)
- net 29: now also J18.8 (Pin_8)
- net BLDC_PWM: now also J7.3 (Pin_3); no longer J7.1 (Pin_1)
- net GND: now also J1.1 (Pin_1), J2.1 (Pin_1), J7.1 (Pin_1), C11.2, J14.2 (Ext), J16.1 (Pin_1), J17.1 (Pin_1), J18.1 (Pin_1); no longer J1.3 (Pin_3), J2.3 (Pin_3), J7.3 (Pin_3)
- net I2C_SCL1: now also J16.2 (Pin_2)
- net I2C_SDA1: now also J16.3 (Pin_3)
- net at BT1.1 (+), C3.1, U3.6 (V_BCKP): now also R11.2
- net at U3.11 (RF_IN): now also J14.1 (In)
- net TIMEPULSE: now reaches U3.4 (TIMEPULSE)
- net EXTINT: now reaches U3.5 (EXTINT)
- net 20 renamed clutch1
- net clutch1: now also J17.3 (Pin_3)
- net 21 renamed clutch2
- net clutch2: now also J17.2 (Pin_2)
- new net: D1.1 (K), R11.1
- new net temp1: J2.2 (Pin_2), R2.1, U1.9 (OUT1C)
- new net temp2: J1.2 (Pin_2), R1.1, U1.39 (A15)
- no-connect marks 18 -> 22
Other:
- moved on the sheet: J1, J2, R1, R2
