File: Hardware/Tim/main_board2.0/winderboard_2.0/winderboard_2.0.kicad_pcb (KiCad board)
At the start: 2 copper layers, 20.3 x 26.7 mm, 55 parts, among them J1 Conn_01x03_Socket, J10 Conn_01x04_Socket, J11 Conn_01x06_Socket, J12 Conn_01x04_Socket, J13 Conn_01x02_Socket, J14 Conn_01x10_Pin, J15 Conn_01x04_Pin, J2 Conn_01x03_Socket, J3 Conn_01x02_Socket, J4 Conn_01x02_Socket, J5 Conn_01x05_Socket, J6 Conn_01x05_Socket, J7 Conn_01x03_Socket, J8 Conn_01x02_Socket, J9 Conn_01x02_Socket, M1 Stepper_Motor_bipolar, M2 Motor_Servo, Q1 NMOS, Q2 NMOS, Q3 DMN6040SK3-13, U1 DEV-16771, U2 MS5607-02BA, U3 MAX-M10S, U4 TMP100, U5 LM1084-ADJ, U6 0.3 Ohm Resistor, U7 INA260, U8 TPS62133

Commit message: First draft of final
Parts:
- removed C2: 100nF, Capacitor_SMD:C_0603_1608Metric_Pad1.08x0.95mm_HandSolder
- removed C6, C7: 0.1uF, Capacitor_SMD:C_0603_1608Metric_Pad1.08x0.95mm_HandSolder
- removed R7, R8: 4.7k, Resistor_SMD:R_0603_1608Metric_Pad0.98x0.95mm_HandSolder
- removed U4: TMP100, Package_TO_SOT_SMD:SOT-23-6
- removed U7: INA260, Package_SO:TSSOP-16_4.4x5mm_P0.65mm
- added C11: 22uF, Capacitor_SMD:C_0603_1608Metric_Pad1.08x0.95mm_HandSolder, F.Cu at (200.3, 137.0)
- added D1: D_Schottky, Diode_SMD:D_SOD-123F, F.Cu at (203.8, 59.8)
- added G***: LOGO, Aesthetics:logosmall, F.Cu at (211.9, 76.3)
- added J16: INA260, Connector_JST:JST_XH_B4B-XH-A_1x04_P2.50mm_Vertical, B.Cu at (219.5, 130.2)
- added J17: Conn_01x04_Socket, Connector_JST:JST_XH_B4B-XH-A_1x04_P2.50mm_Vertical, B.Cu at (162.8, 127.2)
- added J18: Conn_01x08_Pin, Connector_PinHeader_2.54mm:PinHeader_1x08_P2.54mm_Vertical, B.Cu at (208.2, 108.2)
- added J19: Conn_01x01_Pin, MountingHole:MountingHole_3.2mm_M3_DIN965_Pad, F.Cu at (219.0, 152.0)
- added J19: Conn_01x01_Pin, MountingHole:MountingHole_3.2mm_M3_DIN965_Pad, F.Cu at (162.8, 152.0)
- added J19: Conn_01x01_Pin, MountingHole:MountingHole_3.2mm_M3_DIN965_Pad, F.Cu at (162.8, 47.0)
- added J19: Conn_01x01_Pin, MountingHole:MountingHole_3.2mm_M3_DIN965_Pad, F.Cu at (219.0, 47.0)
- added R11: 3.3k, Resistor_SMD:R_0603_1608Metric_Pad0.98x0.95mm_HandSolder, F.Cu at (201.7, 59.2)
- A1, BT3, J13, RV1, U1: moved to B.Cu
- BT2: value BAT-HLD-001 -> RTC Battery; moved to B.Cu
- J1: value Conn_01x03_Socket -> Temp Probe 1; footprint Connector_JST:JST_EH_B3B-EH-A_1x03_P2.50mm_Vertical -> Connector_JST:JST_XH_B3B-XH-A_1x03_P2.50mm_Vertical; moved to B.Cu
- J10: value Conn_01x04_Socket -> XBee Explorer; moved to B.Cu
- J11: value Conn_01x06_Socket -> BNO055; moved to B.Cu
- J12: value Conn_01x04_Socket -> IR Temp Sensor; footprint Connector_JST:JST_EH_B4B-EH-A_1x04_P2.50mm_Vertical -> Connector_JST:JST_XH_B4B-XH-A_1x04_P2.50mm_Vertical; moved to B.Cu
- J14: value Conn_01x10_Pin -> Conn_Coaxial; footprint Connector_PinHeader_2.54mm:PinHeader_1x10_P2.54mm_Vertical -> Connector_Coaxial:U.FL_Molex_MCRF_73412-0110_Vertical
- J15: value Conn_01x04_Pin -> I2C Pinout; moved to B.Cu
- J2: value Conn_01x03_Socket -> Temp Probe 2; footprint Connector_JST:JST_EH_B3B-EH-A_1x03_P2.50mm_Vertical -> Connector_JST:JST_XH_B3B-XH-A_1x03_P2.50mm_Vertical; moved to B.Cu
- J3: value Conn_01x02_Socket -> Limit Switch 2; moved to B.Cu
- J4: value Conn_01x02_Socket -> Limit Switch 1; moved to B.Cu
- J5: value Conn_01x05_Socket -> Encoder 1; footprint Connector_JST:JST_XH_B5B-XH-AM_1x05_P2.50mm_Vertical -> Connector_JST:JST_XH_B5B-XH-A_1x05_P2.50mm_Vertical; moved to B.Cu
- J6: value Conn_01x05_Socket -> Encoder 2; footprint Connector_JST:JST_XH_B5B-XH-AM_1x05_P2.50mm_Vertical -> Connector_JST:JST_XH_B5B-XH-A_1x05_P2.50mm_Vertical; moved to B.Cu
- J7: value Conn_01x03_Socket -> ESC; footprint Connector_JST:JST_EH_B3B-EH-A_1x03_P2.50mm_Vertical -> Connector_JST:JST_XH_B3B-XH-A_1x03_P2.50mm_Vertical; moved to B.Cu
- J8: value Conn_01x02_Socket -> Heater 1; moved to B.Cu
- J9: value Conn_01x02_Socket -> Heater 2; moved to B.Cu
- M1: footprint Connector_JST:JST_EH_B4B-EH-A_1x04_P2.50mm_Vertical -> Connector_JST:JST_XH_B4B-XH-A_1x04_P2.50mm_Vertical; moved to B.Cu
- M2: footprint Connector_JST:JST_EH_B3B-EH-A_1x03_P2.50mm_Vertical -> Connector_JST:JST_XH_B3B-XH-A_1x03_P2.50mm_Vertical; moved to B.Cu
- R5, R6: value R_Small -> ??
- moved J14 186.3 mm to (219.4, 53.8)
- moved R5 168.0 mm to (209.9, 64.2), turned to 180 degrees
- moved U3 165.4 mm to (210.9, 57.4), turned to 90 degrees
- moved U5 164.0 mm to (209.7, 128.9)
- moved J10 163.2 mm to (187.8, 85.5), turned to 180 degrees
- moved C8 159.7 mm to (203.2, 143.6)
- moved C1 159.5 mm to (214.6, 64.2)
- moved C9 158.2 mm to (203.9, 141.0), turned to -90 degrees
- moved C10 155.8 mm to (203.9, 137.5), turned to 90 degrees
- moved J8 149.9 mm to (171.2, 144.6), turned to 90 degrees
- moved C5 147.1 mm to (194.7, 130.7), turned to 180 degrees
- moved C3 145.9 mm to (200.0, 59.2), turned to -90 degrees
- moved U6 143.6 mm to (198.2, 117.1), turned to 180 degrees
- moved R3 143.4 mm to (203.0, 91.2), turned to 180 degrees
- moved C4 143.3 mm to (198.0, 95.0), turned to -90 degrees
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Connections:
- C1 pad 1: temp1 -> +3.3V
- C4 pad 1: temp1 -> +3.3V
- J1 pad 1: Net-(J1-Pin_1) -> GND
- J1 pad 2: temp1 -> temp2
- J1 pad 3: GND -> +3.3V
- J14 pad 1: 10 -> Net-(J14-In)
- J14 pad 2: 11 -> GND
- J2 pad 1: Net-(J2-Pin_1) -> GND
- J2 pad 3: GND -> +3.3V
- J7 pad 1: BLDC_PWM -> GND
- J7 pad 3: GND -> BLDC_PWM
- R1 pad 1: temp1 -> temp2
- R1 pad 2: Net-(J1-Pin_1) -> +3.3V
- R2 pad 2: Net-(J2-Pin_1) -> +3.3V
- R3 pad 1: temp1 -> +3.3V
- R4 pad 1: temp1 -> +3.3V
- U1 pad 20: 20 -> clutch1
- U1 pad 21: 21 -> clutch2
- U1 pad 26: 26 -> EXTINT
- U1 pad 27: 27 -> TIMEPULSE
- U1 pad 3.3V_1: temp1 -> +3.3V
- U1 pad 3.3V_2: temp1 -> +3.3V
- U1 pad 3.3V_3: temp1 -> +3.3V
- U1 pad 39: temp1 -> temp2
- U2 pad 1: temp1 -> +3.3V
- U2 pad 2: temp1 -> +3.3V
- U3 pad 11: unconnected-(U3-RF_IN-Pad11) -> Net-(J14-In)
- U3 pad 4: unconnected-(U3-TIMEPULSE-Pad4) -> TIMEPULSE
- U3 pad 5: unconnected-(U3-EXTINT-Pad5) -> EXTINT
- U3 pad 7: temp1 -> +3.3V
- U3 pad 8: temp1 -> +3.3V
Routing:
- net +3.3V: track 0.00 -> 139.0 mm, vias 0 -> 7
- net cutdown: track 0.00 -> 72.1 mm, vias 0 -> 3
- net clutch1: track 0.00 -> 68.0 mm, vias 0 -> 1
- net clutch2: track 0.00 -> 67.8 mm
- net stepper_sleep: track 0.00 -> 67.6 mm, vias 0 -> 4
- net I2C_SDA1: track 0.00 -> 66.4 mm, vias 0 -> 3
- net IR_SCL: track 0.00 -> 63.8 mm, vias 0 -> 1
- net stepper_step: track 0.00 -> 63.7 mm, vias 0 -> 1
- net stepper_dir: track 0.00 -> 63.1 mm, vias 0 -> 1
- net EXTINT: track 0.00 -> 61.9 mm, vias 0 -> 2
- net I2C_SCL1: track 0.00 -> 61.9 mm, vias 0 -> 2
- net TIMEPULSE: track 0.00 -> 58.3 mm, vias 0 -> 2
- net RTC_Batt: track 0.00 -> 55.2 mm, vias 0 -> 7
- net stepper_MS1: track 0.00 -> 53.1 mm, vias 0 -> 1
- net stepper_MS2: track 0.00 -> 52.7 mm, vias 0 -> 1
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- added copper zone on F.Cu, net +5V
- added copper zone on In2.Cu, net +5V
- added copper zone on F.Cu, net +BATT
- added copper zone on In2.Cu, net +BATT
- added copper zone on B.Cu, net GND
- added copper zone on F.Cu, net GND
- added copper zone on In1.Cu, net GND
- added copper zone on F.Cu, net Net-(J13-Pin_2)
- added copper zone on F.Cu, net Net-(L1-Pad1)
- added copper zone on F.Cu, net Net-(U5-VO)
- added copper zone on B.Cu, net RTC_Batt
Other:
- board size 20.3 x 26.7 mm -> 63.8 x 113 mm
- copper layers 2 -> 4
- board text added: "By Akemi, JJ, and Shipman"
- board text added: "UMD BPP Bobot-2 Board"

Commit message: minor changes, more needed
Routing:
- net +3.3V: track 139.0 -> 158.5 mm
- net GND: track 30.3 -> 29.5 mm
