File: Hardware/Tim/main_board2.0/winderboard_2.0/winderboard_2.0.kicad_pcb (KiCad board)
At the start: 4 copper layers, 63.8 x 113 mm, 59 parts, among them J1 Temp Probe 1, J10 XBee Explorer, J11 BNO055, J12 IR Temp Sensor, J13 Conn_01x02_Socket, J14 Conn_Coaxial, J15 I2C Pinout, J16 INA260, J17 Conn_01x04_Socket, J18 Conn_01x08_Pin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

Commit message: recovered from covid push
Parts:
- moved U6 0.05 mm to (198.3, 117.1)
Routing:
- net stepper_MS1: track 53.1 -> 51.7 mm
- net stepper_MS2: track 52.7 -> 52.1 mm
- net stepper_MS3: track 51.8 -> 51.2 mm
